File: pcbs/FTDI/1.0/FTDI.kicad_pcb (KiCad board)
At the start: 2 copper layers, 85 x 55 mm, 30 parts, among them J1 Conn_01x04_Pin, J2 Conn_01x04_Pin, J5 Conn_01x03_Pin, Q1 2N3055, Q2 2N3055, U1 FT232RL, U2 ADUM3160

Commit message: Updates
Parts:
- added J3: Conn_01x02_Pin, Connector_PinHeader_2.54mm:PinHeader_1x02_P2.54mm_Vertical, F.Cu at (127.4, 98.4)
- added J4: Conn_01x02_Pin, Connector_PinHeader_2.54mm:PinHeader_1x02_P2.54mm_Vertical, F.Cu at (151.6, 98.5)
- added R6: 4.7K, Resistor_SMD:R_0603_1608Metric_Pad0.98x0.95mm_HandSolder, F.Cu at (124.3, 99.7)
- added R7: 4.7K, Resistor_SMD:R_0603_1608Metric_Pad0.98x0.95mm_HandSolder, F.Cu at (154.8, 99.8)
- moved C10 2.61 mm to (153.4, 69.9)
- moved C11 2.61 mm to (160.8, 69.9)
Connections:
- U2 pad 13: 5V -> SPD
- U2 pad 5: USB_VBUS -> SPU
Routing:
- net SPU: track 0.00 -> 11.5 mm
- net SPD: track 0.00 -> 10.6 mm
- net 3V3: track 120.8 -> 130.1 mm
- net RTS: track 12.3 -> 17.3 mm
- net D-: track 29.5 -> 34.0 mm
- net USB_VBUS: track 31.7 -> 35.6 mm, vias 1 -> 2
- net RX: track 28.6 -> 30.9 mm
- net TX: track 31.8 -> 33.8 mm, vias 2 -> 1
- net 5V: track 125.5 -> 123.5 mm, vias 2 -> 6
- net USB_GND: track 40.6 -> 42.1 mm, vias 0 -> 4
- net GND: track 1.36 -> 0.00 mm, vias 4 -> 2
- net USB_D+: track 28.6 -> 27.7 mm
- net Net-(Q2-B): track 10.6 -> 11.4 mm
- net DTR: track 22.1 -> 21.8 mm, vias 4 -> 2
- net BOOT: track 27.5 -> 27.6 mm, vias 0 -> 1
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Other:
- board text added: "LOW_SPD"
