File: pcbs/FTDI/1.0/FTDI.kicad_sch (KiCad schematic)
At the start: 30 parts, among them J1 Conn_01x04_Pin, J2 Conn_01x04_Pin, J5 Conn_01x03_Pin, Q1 2N3055, Q2 2N3055, U1 FT232RL, U2 ADUM3160

Commit message: Updates
Parts:
- added J3, J4: Conn_01x02_Pin, Connector_PinHeader_2.54mm:PinHeader_1x02_P2.54mm_Vertical, symbol Connector:Conn_01x02_Pin
- added R6, R7: 4.7K, Resistor_SMD:R_0603_1608Metric_Pad0.98x0.95mm_HandSolder, symbol Device:R_Small
- R1: value 100R -> 150R
Connections:
- net 5V: now also R6.1; no longer U2.13 (SPD)
- net GND: now also J3.2 (Pin_2), J4.2 (Pin_2)
- net USB_VBUS: now also R7.1; no longer U2.5 (SPU)
- new net SPD: J3.1 (Pin_1), R6.2, U2.13 (SPD)
- new net SPU: J4.1 (Pin_1), R7.2, U2.5 (SPU)
Other:
- moved on the sheet: C1, C10, C11, C2, C3, C4, C5, D1, D2, H1, H2, H3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
