File: pcbs/input-sel/0.3/input-sel.kicad_pcb (KiCad board)
At the start: 2 copper layers, 85 x 55 mm, 46 parts, among them J1 Conn_01x03_Pin, J10 Conn_01x02_Male, J2 Conn_01x03_Pin, J3 Conn_01x03_Pin, J4 Conn_01x03_Pin, J5 Conn_01x03_Pin, J6 Conn_01x03_Pin, J7 Conn_01x03_Male, J8 Conn_01x03_Pin, J9 Conn_01x04_Pin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

Commit message: Updates
Parts:
- moved C5 11.3 mm to (127.0, 73.2)
- moved C2 11.2 mm to (96.4, 73.2)
- moved C6 10.9 mm to (137.1, 70.3)
- moved C3 10.9 mm to (106.6, 70.3)
- moved C8 9.90 mm to (116.8, 70.3)
- moved C11 9.88 mm to (147.3, 70.3)
- moved C7 9.41 mm to (106.6, 73.2)
- moved C10 9.39 mm to (137.1, 73.2)
- moved C12 0.82 mm to (147.3, 73.2)
- moved C9 0.80 mm to (116.8, 73.2)
- moved C4 0.79 mm to (127.0, 70.3)
- moved C1 0.76 mm to (96.4, 70.3)
Connections:
- C1 pad 1: RCA1_R -> RCA1_L
- C1 pad 2: Net-(U1-IN1R) -> Net-(U1-IN2L)
- C10 pad 1: RCA4_L -> RCA5_R
- C10 pad 2: Net-(U2-IN1L) -> Net-(U2-IN3R)
- C11 pad 1: RCA5_L -> RCA6_L
- C11 pad 2: Net-(U2-IN2L) -> Net-(C11-Pad2)
- C12 pad 1: RCA6_L -> RCA6_R
- C12 pad 2: Net-(U2-IN3L) -> Net-(C12-Pad2)
- C14 pad 2: GND -> AGND
- C15 pad 2: GND -> AGND
- C16 pad 2: GND -> AGND
- C17 pad 1: GND -> AGND
- C2 pad 1: RCA2_R -> RCA1_R
- C20 pad 1: GND -> AGND
- C22 pad 2: GND -> AGND
- C3 pad 1: RCA3_R -> RCA2_L
- C3 pad 2: Net-(U1-IN3R) -> Net-(U1-IN3L)
- C4 pad 1: RCA4_R -> RCA4_L
- C4 pad 2: Net-(U2-IN1R) -> Net-(U2-IN2L)
- C5 pad 1: RCA5_R -> RCA4_R
- C6 pad 1: RCA6_R -> RCA5_L
- C6 pad 2: Net-(U2-IN3R) -> Net-(U2-IN3L)
- C7 pad 1: RCA1_L -> RCA2_R
- C7 pad 2: Net-(U1-IN1L) -> Net-(U1-IN3R)
- C8 pad 1: RCA2_L -> RCA3_L
- C8 pad 2: Net-(U1-IN2L) -> Net-(U2-IN1L)
- C9 pad 1: RCA3_L -> RCA3_R
- C9 pad 2: Net-(U1-IN3L) -> Net-(U2-IN1R)
- D1 pad 1: GND -> AGND
- R1 pad 1: GND -> AGND
- R2 pad 1: GND -> AGND
- R3 pad 1: GND -> AGND
- R5 pad 1: GND -> AGND
- U1 pad 1: Net-(U1-IN1L) -> AGND
- U1 pad 16: GND -> AGND
- U1 pad 6: Net-(U1-IN1R) -> AGND
- U2 pad 16: GND -> AGND
- U2 pad 5: GND -> Net-(C11-Pad2)
- U2 pad 8: GND -> Net-(C12-Pad2)
Routing:
- net AGND: track 0.00 -> 246.6 mm, vias 0 -> 11
- net Net-(U1-IN1R): track 41.6 -> 0.00 mm, vias 2 -> 0
- net Net-(C11-Pad2): track 0.00 -> 31.1 mm, vias 0 -> 2
- net Net-(U1-IN1L): track 28.6 -> 0.00 mm, vias 2 -> 0
- net Net-(C12-Pad2): track 0.00 -> 27.3 mm, vias 0 -> 2
- net Net-(U1-IN2R): track 30.2 -> 48.3 mm
- net Net-(U2-IN3L): track 34.1 -> 17.6 mm
- net Net-(U1-IN2L): track 22.9 -> 37.7 mm
- net Net-(U2-IN1L): track 22.9 -> 36.3 mm
- net V+: track 86.1 -> 98.7 mm
- net Net-(U1-OUTL): track 32.1 -> 20.2 mm, vias 2 -> 0
- net EXPAND_L: track 42.7 -> 52.0 mm
- net Net-(U2-IN1R): track 28.8 -> 37.6 mm
- net Net-(U2-OUTL): track 25.2 -> 33.9 mm
- net Net-(U2-IN2R): track 22.6 -> 29.8 mm
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- added copper zone on F.Cu, net AGND
- removed copper zone on F.Cu, net GND
