File: pcbs/input-sel/0.3/input-sel.kicad_sch (KiCad schematic)
At the start: 46 parts, among them J1 Conn_01x03_Pin, J10 Conn_01x02_Male, J2 Conn_01x03_Pin, J3 Conn_01x03_Pin, J4 Conn_01x03_Male, J4 Conn_01x03_Pin, J5 Conn_01x03_Pin, J6 Conn_01x03_Pin, J8 Conn_01x03_Pin, J9 Conn_01x04_Pin, U1 NJM2750, U2 NJM2750

Commit message: Updates
Connections:
- net AGND: now also C14.2, C15.2, C16.2, C17.1, C20.1, C22.2, D1.1 (K), R1.1, R2.1, R3.1, R5.1, U1.1 (IN1L), U1.16 (GND), U1.6 (IN1R), U2.16 (GND)
- net RCA1_L: now also C1.1; no longer C7.1
- net RCA1_R: now also C2.1; no longer C1.1
- net RCA2_L: now also C3.1; no longer C8.1
- net RCA2_R: now also C7.1; no longer C2.1
- net RCA3_L: now also C8.1; no longer C9.1
- net RCA3_R: now also C9.1; no longer C3.1
- net RCA4_L: now also C4.1; no longer C10.1
- net RCA4_R: now also C5.1; no longer C4.1
- net RCA5_L: now also C6.1; no longer C11.1
- net RCA5_R: now also C10.1; no longer C5.1
- net RCA6_L: now also C11.1; no longer C12.1
- net RCA6_R: now also C12.1; no longer C6.1
- net at C6.2: now also U2.13 (IN3L); no longer U2.9 (IN3R)
- net at C4.2: now also U2.3 (IN2L); no longer U2.6 (IN1R)
- net at C12.2: now also U2.8 (IN4L); no longer U2.13 (IN3L)
- net at C10.2: now also U2.9 (IN3R); no longer U2.1 (IN1L)
- net at U1.3 (IN2L): now also C1.2; no longer C8.2
- net at C7.2: now also U1.9 (IN3R); no longer U1.1 (IN1L)
- net at U1.13 (IN3L): now also C3.2; no longer C9.2
- net at C11.2: now also U2.5 (IN4L); no longer U2.3 (IN2L)
- removed net GND: C14.2, C15.2, C16.2, C17.1, C20.1, C22.2, D1.1 (K), R1.1, R2.1, R3.1, R5.1, U1.16 (GND), U2.16 (GND), U2.5 (IN4L), U2.8 (IN4L)
- new net: C9.2, U2.6 (IN1R)
- new net: C8.2, U2.1 (IN1L)
Other:
- moved on the sheet: C22, D1, R4
