File: pcbs/uproc/1.0/uproc.kicad_sch (KiCad schematic)
At the start: 68 parts, among them J1 Conn_01x02_Male, J10 Conn_01x02_Male, J11 Conn_01x02_Male, J12 Conn_01x02_Male, J13 Conn_01x03_Pin, J14 Conn_01x05_Pin, J15 Conn_01x04_Pin, J16 Conn_01x02_Male, J17 Conn_01x05_Pin, J18 Conn_01x02_Male, J19 Conn_01x02_Male, J2 Conn_01x05_Pin, J3 Conn_01x04_Pin, J4 Conn_01x03_Pin, J5 Conn_01x02_Male, J6 Conn_01x04_Pin, J7 Conn_01x02_Male, J8 Conn_01x02_Male, J9 Conn_01x02_Male, Q1 BC817, Q2 BC817, U1 TMP100, U3 TCA9517DR, U4 ESP32-S3-WROOM-1

Commit message: Updates
Parts:
- added J19: Conn_01x04_Pin, Connector_JST:JST_PH_B4B-PH-K_1x04_P2.00mm_Vertical, symbol Connector:Conn_01x04_Pin
- renumbered C7 to C1, C6 to C10, C5 to C11, C8 to C12, C1 to C2, C2 to C4, C9 to C5, C10 to C6, C11 to C7, C12 to C8, C4 to C9, H3 to H2, H2 to H3, J4 to J1, J9 to J10, J16 to J11, J17 to J12, J3 to J13, J19 to J14, J11 to J15, J8 to J16, J6 to J17, J12 to J18, J7 to J2, J13 to J20, J10 to J3, J18 to J4, J1 to J5, J5 to J6, J2 to J7, J14 to J8, J15 to J9, R17 to R1, R8 to R10, R22 to R11, R21 to R12, R23 to R13, R16 to R14, R10 to R15, R13 to R16, R2 to R17, R3 to R18, R4 to R19, R1 to R2, R5 to R20, R6 to R21, R15 to R22, R7 to R23, R14 to R24, R24 to R3, R18 to R4, R11 to R5, R19 to R6, R9 to R7, R20 to R8, R12 to R9, U4 to U1, U3 to U2, U1 to U3
Connections:
- net SPI_CLK: now also J19.3 (Pin_3)
- net SPI_MOSI: now also J19.1 (Pin_1), J19.2 (Pin_2)
- net SPI_CS2: now reaches U1.31 (GPIO38/FSPIWP/SUBSPIWP)
- net SPI_CS2: now also J19.4 (Pin_4)
Other:
- moved on the sheet: C11, C13, C2, C3, C4, C5, C6, C7, C8, C9, D1, D2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
