File: pcbs/uproc/1.0/uproc.kicad_sch (KiCad schematic)
At the start: 69 parts, among them J1 Conn_01x03_Pin, J10 Conn_01x02_Male, J11 Conn_01x02_Male, J12 Conn_01x05_Pin, J13 Conn_01x04_Pin, J14 Conn_01x02_Male, J15 Conn_01x02_Male, J16 Conn_01x02_Male, J17 Conn_01x04_Pin, J18 Conn_01x02_Male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

Commit message: Updates to pcbs
Parts:
- R15, R16, R22, R24: value 10K -> 4.7K
Changed lines of the file:
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@@
 			)
 		)
-		(property "Value" "10K"
+		(property "Value" "4.7K"
 			(at 60.96 36.8299 0)
 			(effects
@@
 			)
 		)
-		(property "Value" "10K"
+		(property "Value" "4.7K"
 			(at 49.149 31.7499 0)
 			(effects
@@
 			)
 		)
-		(property "Value" "10K"
+		(property "Value" "4.7K"
 			(at 69.469 38.0999 0)
 			(effects
@@
 			)
 		)
-		(property "Value" "10K"
+		(property "Value" "4.7K"
 			(at 40.64 30.4799 0)
 			(effects
