File: pcbs/uproc/1.0/uproc.kicad_pcb (KiCad board)
At the start: 2 copper layers, 85 x 55 mm, 68 parts, among them J1 Conn_01x02_Male, J10 Conn_01x02_Male, J11 Conn_01x02_Male, J12 Conn_01x02_Male, J13 Conn_01x03_Pin, J14 Conn_01x05_Pin, J15 Conn_01x04_Pin, J16 Conn_01x02_Male, J17 Conn_01x05_Pin, J18 Conn_01x02_Male, J19 Conn_01x02_Male, J2 Conn_01x05_Pin, J3 Conn_01x04_Pin, J4 Conn_01x03_Pin, J5 Conn_01x02_Male, J6 Conn_01x04_Pin, J7 Conn_01x02_Male, J8 Conn_01x02_Male, J9 Conn_01x02_Male, Q1 BC817, Q2 BC817, U1 TMP100, U3 TCA9517DR, U4 ESP32-S3-WROOM-1

Commit message: Updates
Parts:
- added J19: Conn_01x04_Pin, Connector_JST:JST_PH_B4B-PH-K_1x04_P2.00mm_Vertical, F.Cu at (170.4, 99.0)
- moved J16 19.5 mm to (165.6, 66.3), turned to 180 degrees
- moved R22 9.51 mm to (154.9, 86.5), turned to -90 degrees
- moved J10 8.28 mm to (135.9, 90.8)
- moved R14 8.28 mm to (141.4, 90.8)
- moved R24 7.90 mm to (156.7, 86.5), turned to -90 degrees
- moved J15 6.67 mm to (162.9, 86.1)
- moved U2 6.65 mm to (149.1, 91.6)
- moved C10 6.65 mm to (150.9, 95.5)
- moved C9 6.65 mm to (150.9, 87.7)
- moved J18 6.57 mm to (170.4, 86.1)
- moved R15 4.49 mm to (149.7, 79.3)
- moved R16 4.49 mm to (149.7, 81.2)
- moved C11 3.01 mm to (160.2, 77.6)
- moved U3 3.01 mm to (160.1, 74.4)
- moved C4 2.95 mm to (117.5, 70.7)
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- renumbered C7 to C1, C6 to C10, C5 to C11, C8 to C12, C1 to C2, C2 to C4, C9 to C5, C10 to C6, C11 to C7, C12 to C8, C4 to C9, H3 to H2, H2 to H3, J4 to J1, J9 to J10, J16 to J11, J17 to J12, J3 to J13, J19 to J14, J11 to J15, J8 to J16, J6 to J17, J12 to J18, J7 to J2, J13 to J20, J10 to J3, J18 to J4, J1 to J5, J5 to J6, J2 to J7, J14 to J8, J15 to J9, R17 to R1, R8 to R10, R22 to R11, R21 to R12, R23 to R13, R16 to R14, R10 to R15, R13 to R16, R2 to R17, R3 to R18, R4 to R19, R1 to R2, R5 to R20, R6 to R21, R15 to R22, R7 to R23, R14 to R24, R24 to R3, R18 to R4, R11 to R5, R19 to R6, R9 to R7, R20 to R8, R12 to R9, U4 to U1, U3 to U2, U1 to U3
Connections:
- U1 pad 31: unconnected-(U4-GPIO38/FSPIWP/SUBSPIWP-Pad31) -> SPI_CS2
Routing:
- net SPI_MOSI: track 39.2 -> 111.0 mm, vias 2 -> 4
- net SPI_CS2: track 0.00 -> 50.1 mm, vias 0 -> 2
- net SPI_CLK: track 47.8 -> 88.9 mm, vias 2 -> 0
- net ENABLE: track 125.6 -> 102.6 mm, vias 1 -> 3
- net 5V: track 158.5 -> 139.4 mm, vias 2 -> 4
- net Net-(D2-A): track 20.7 -> 4.00 mm
- net GND: track 384.3 -> 399.6 mm, vias 14 -> 21
- net 3V3: track 260.8 -> 251.2 mm, vias 5 -> 7
- net SDA: track 100.1 -> 107.0 mm, vias 3 -> 5
- net INPUT_CH2: track 52.3 -> 58.9 mm
- net SPI_CS: track 46.6 -> 40.0 mm
- net TX: track 33.4 -> 39.7 mm, vias 0 -> 3
- net SCL: track 105.6 -> 100.0 mm, vias 2 -> 5
- net INPUT_BUTTON: track 46.5 -> 50.9 mm
- net INPUT_CH1: track 52.0 -> 56.4 mm
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Other:
- board text added: "SPI"

Commit message: Updates to pcbs
Parts:
- R15, R16, R22, R24: value 10K -> 4.7K
Routing:
- net SPI_CLK: track 88.9 -> 88.3 mm
