File: pcbs/ADC/1.0/ADC.kicad_sch (KiCad schematic)
At the start: 45 parts, among them J1 Conn_01x04_Pin, J3 Conn_01x02_Male, J4 Conn_01x03_Pin, J5 Conn_01x03_Pin, J9 Conn_01x04_Pin, U1 ZLDO1117QG33TA, U2 PCM1863, Y1 24.576 MHz

Commit message: Updating PCBs
Parts:
- Y1: Mouser (none) -> 520-245.7-8-33-RWYT
- renumbered C20 to C1, C4 to C10, C18 to C11, C19 to C12, C10 to C13, C11 to C14, C12 to C15, C13 to C16, C14 to C18, C15 to C19, C1 to C2, C16 to C20, C2 to C3, C6 to C4, C7 to C6, C8 to C7, C3 to C8, J3 to J2, J4 to J3, J9 to J4, R3 to R1, R8 to R2, R9 to R3, R1 to R4, R7 to R5, R2 to R7, R5 to R8, R4 to R9
Changed lines of the file:
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@@
 		(dnp no)
 		(fields_autoplaced yes)
-		(property "Reference" "C12"
+		(property "Reference" "C15"
 			(at 257.81 41.9162 0)
 			(effects
@@
 			(project "ADC"
 				(path "/ad933f83-dd94-4dcc-b4f2-96fd54138c43"
-					(reference "C12")
+					(reference "C15")
 					(unit 1)
 				)
@@
 			)
 		)
+		(property "Mouser" "520-245.7-8-33-RWYT"
+			(at 99.06 111.76 0)
+			(effects
+				(font
+					(size 1.27 1.27)
+				)
+				(hide yes)
+			)
+		)
 		(pin "4"
 		)
@@
 		(dnp no)
 		(fields_autoplaced yes)
-		(property "Reference" "R7"
+		(property "Reference" "R5"
 			(at 256.54 96.52 90)
 			(effects
@@
 			(project "ADC"
 				(path "/ad933f83-dd94-4dcc-b4f2-96fd54138c43"
-					(reference "R7")
+					(reference "R5")
 					(unit 1)
 				)
@@
 		(dnp no)
 		(fields_autoplaced yes)
-		(property "Reference" "C14"
+		(property "Reference" "C18"
 			(at 180.34 78.7462 0)
 			(effects
@@
 			(project "ADC"
 				(path "/ad933f83-dd94-4dcc-b4f2-96fd54138c43"
-					(reference "C14")
+					(reference "C18")
 					(unit 1)
 				)
@@
 		(dnp no)
 		(fields_autoplaced yes)
-		(property "Reference" "J3"
+		(property "Reference" "J2"
 			(at 57.912 64.7701 0)
 			(effects
@@
 			(project "ChannelSelector"
 				(path "/ad933f83-dd94-4dcc-b4f2-96fd54138c43"
-					(reference "J3")
+					(reference "J2")
 					(unit 1)
 				)
@@
 		(dnp no)
 		(fields_autoplaced yes)
-		(property "Reference" "C4"
+		(property "Reference" "C10"
 			(at 162.814 37.2999 0)
 			(effects
@@
 			(project "ChannelSelector"
 				(path "/ad933f83-dd94-4dcc-b4f2-96fd54138c43"
-					(reference "C4")
+					(reference "C10")
 					(unit 1)
 				)
@@
 		(dnp no)
 		(fields_autoplaced yes)
-		(property "Reference" "R8"
+		(property "Reference" "R2"
 			(at 96.52 29.2099 0)
 			(effects
@@
 			(project "ADC"
 				(path "/ad933f83-dd94-4dcc-b4f2-96fd54138c43"
-					(reference "R8")
+					(reference "R2")
 					(unit 1)
 				)
@@
 		(dnp no)
 		(fields_autoplaced yes)
-		(property "Reference" "R5"
+		(property "Reference" "R8"
 			(at 166.37 88.9 90)
 			(effects
@@
 			(project "ADC"
 				(path "/ad933f83-dd94-4dcc-b4f2-96fd54138c43"
-					(reference "R5")
+					(reference "R8")
 					(unit 1)
 				)
@@
 		(dnp no)
 		(fields_autoplaced yes)
-		(property "Reference" "C1"
+		(property "Reference" "C2"
 			(at 34.671 111.7536 0)
 			(effects
@@
 			(project "ADC"
 				(path "/ad933f83-dd94-4dcc-b4f2-96fd54138c43"
-					(reference "C1")
+					(reference "C2")
 					(unit 1)
 				)
@@
 		(dnp no)
 		(fields_autoplaced yes)
-		(property "Reference" "C19"
+		(property "Reference" "C12"
 			(at 85.09 113.0362 0)
 			(effects
@@
 			(project "ADC"
 				(path "/ad933f83-dd94-4dcc-b4f2-96fd54138c43"
-					(reference "C19")
+					(reference "C12")
 					(unit 1)
 				)
@@
 		(dnp no)
 		(fields_autoplaced yes)
-		(property "Reference" "C8"
+		(property "Reference" "C7"
 			(at 284.48 41.9162 0)
 			(effects
@@
 			(project "ADC"
 				(path "/ad933f83-dd94-4dcc-b4f2-96fd54138c43"
-					(reference "C8")
+					(reference "C7")
 					(unit 1)
 				)
@@
 		(dnp no)
 		(fields_autoplaced yes)
-		(property "Reference" "C7"
+		(property "Reference" "C6"
 			(at 294.64 41.9162 0)
 			(effects
@@
 			(project "ADC"
 				(path "/ad933f83-dd94-4dcc-b4f2-96fd54138c43"
-					(reference "C7")
+					(reference "C6")
 					(unit 1)
 				)
@@
 		(dnp no)
 		(fields_autoplaced yes)
-		(property "Reference" "R9"
+		(property "Reference" "R3"
 			(at 109.22 29.2099 0)
 			(effects
@@
 			(project "ADC"
 				(path "/ad933f83-dd94-4dcc-b4f2-96fd54138c43"
-					(reference "R9")
+					(reference "R3")
 					(unit 1)
 				)
@@
 		(on_board yes)
 		(dnp no)
-		(property "Reference" "C16"
+		(property "Reference" "C20"
 			(at 157.48 97.79 90)
 			(effects
@@
 			(project "ADC"
 				(path "/ad933f83-dd94-4dcc-b4f2-96fd54138c43"
-					(reference "C16")
+					(reference "C20")
 					(unit 1)
 				)
@@
 		(dnp no)
 		(fields_autoplaced yes)
-		(property "Reference" "R3"
+		(property "Reference" "R1"
 			(at 83.8488 29.3065 0)
 			(effects
@@
 			(project "ADC"
 				(path "/ad933f83-dd94-4dcc-b4f2-96fd54138c43"
-					(reference "R3")
+					(reference "R1")
 					(unit 1)
 				)
@@
 		(dnp no)
 		(fields_autoplaced yes)
-		(property "Reference" "J9"
+		(property "Reference" "J4"
 			(at 85.725 55.88 0)
 			(effects
@@
 			(project "ADC"
 				(path "/ad933f83-dd94-4dcc-b4f2-96fd54138c43"
-					(reference "J9")
+					(reference "J4")
 					(unit 1)
 				)
@@
 		(dnp no)
 		(fields_autoplaced yes)
-		(property "Reference" "R1"
+		(property "Reference" "R4"
 			(at 248.92 115.57 90)
 			(effects
@@
 			(project "ADC"
 				(path "/ad933f83-dd94-4dcc-b4f2-96fd54138c43"
-					(reference "R1")
+					(reference "R4")
 					(unit 1)
 				)
@@
 		(dnp no)
 		(fields_autoplaced yes)
-		(property "Reference" "C10"
+		(property "Reference" "C13"
 			(at 236.22 41.9162 0)
 			(effects
@@
 			(project "ADC"
 				(path "/ad933f83-dd94-4dcc-b4f2-96fd54138c43"
-					(reference "C10")
+					(reference "C13")
 					(unit 1)
 				)
@@
 		(dnp no)
 		(fields_autoplaced yes)
-		(property "Reference" "C15"
+		(property "Reference" "C19"
 			(at 157.4863 80.01 90)
 			(effects
@@
 			(project "ADC"
 				(path "/ad933f83-dd94-4dcc-b4f2-96fd54138c43"
-					(reference "C15")
+					(reference "C19")
 					(unit 1)
 				)
@@
 		(dnp no)
 		(fields_autoplaced yes)
-		(property "Reference" "J4"
+		(property "Reference" "J3"
 			(at 26.035 58.547 0)
 			(effects
@@
 			(project "InputSel"
 				(path "/ad933f83-dd94-4dcc-b4f2-96fd54138c43"
-					(reference "J4")
+					(reference "J3")
 					(unit 1)
 				)
@@
 		(dnp no)
 		(fields_autoplaced yes)
-		(property "Reference" "C11"
+		(property "Reference" "C14"
 			(at 247.65 41.9162 0)
 			(effects
@@
 			(project "ADC"
 				(path "/ad933f83-dd94-4dcc-b4f2-96fd54138c43"
-					(reference "C11")
+					(reference "C14")
 					(unit 1)
 				)
@@
 		(dnp no)
 		(fields_autoplaced yes)
-		(property "Reference" "C2"
+		(property "Reference" "C3"
 			(at 151.384 37.2999 0)
 			(effects
@@
 			(project "ChannelSelector"
 				(path "/ad933f83-dd94-4dcc-b4f2-96fd54138c43"
-					(reference "C2")
+					(reference "C3")
 					(unit 1)
 				)
@@
 		(dnp no)
 		(fields_autoplaced yes)
-		(property "Reference" "C20"
+		(property "Reference" "C1"
 			(at 173.355 37.2999 0)
 			(effects
@@
 			(project "ADC"
 				(path "/ad933f83-dd94-4dcc-b4f2-96fd54138c43"
-					(reference "C20")
+					(reference "C1")
 					(unit 1)
 				)
@@
 		(dnp no)
 		(fields_autoplaced yes)
-		(property "Reference" "R4"
+		(property "Reference" "R9"
 			(at 166.37 81.28 90)
 			(effects
@@
 			(project "ADC"
 				(path "/ad933f83-dd94-4dcc-b4f2-96fd54138c43"
-					(reference "R4")
+					(reference "R9")
 					(unit 1)
 				)
@@
 		(dnp no)
 		(fields_autoplaced yes)
-		(property "Reference" "C18"
+		(property "Reference" "C11"
 			(at 111.76 113.0362 0)
 			(effects
@@
 			(project "ADC"
 				(path "/ad933f83-dd94-4dcc-b4f2-96fd54138c43"
-					(reference "C18")
+					(reference "C11")
 					(unit 1)
 				)
@@
 		(dnp no)
 		(fields_autoplaced yes)
-		(property "Reference" "R2"
+		(property "Reference" "R7"
 			(at 242.57 101.6 90)
 			(effects
@@
 			(project "ADC"
 				(path "/ad933f83-dd94-4dcc-b4f2-96fd54138c43"
-					(reference "R2")
+					(reference "R7")
 					(unit 1)
 				)
@@
 		(dnp no)
 		(fields_autoplaced yes)
-		(property "Reference" "C13"
+		(property "Reference" "C16"
 			(at 212.09 40.6462 0)
 			(effects
@@
 			(project "ADC"
 				(path "/ad933f83-dd94-4dcc-b4f2-96fd54138c43"
-					(reference "C13")
+					(reference "C16")
 					(unit 1)
 				)
@@
 		(dnp no)
 		(fields_autoplaced yes)
-		(property "Reference" "C3"
+		(property "Reference" "C8"
 			(at 58.801 111.7536 0)
 			(effects
@@
 			(project "ADC"
 				(path "/ad933f83-dd94-4dcc-b4f2-96fd54138c43"
-					(reference "C3")
+					(reference "C8")
 					(unit 1)
 				)
@@
 		(dnp no)
 		(fields_autoplaced yes)
-		(property "Reference" "C6"
+		(property "Reference" "C4"
 			(at 274.32 41.9162 0)
 			(effects
@@
 			(project "ADC"
 				(path "/ad933f83-dd94-4dcc-b4f2-96fd54138c43"
-					(reference "C6")
+					(reference "C4")
 					(unit 1)
 				)

Commit message: Updated screenshots
Parts:
- removed C11, C12: 12n C0G, Capacitor_SMD:C_0805_2012Metric_Pad1.18x1.45mm_HandSolder, symbol Device:C_Small
- removed U3: ~, symbol Custom:PCM1865
- removed Y1: 24.576 MHz, Crystal:Crystal_SMD_3225-4Pin_3.2x2.5mm, symbol Device:Crystal_GND24
- added C1: 0.1u, Capacitor_SMD:C_0805_2012Metric_Pad1.18x1.45mm_HandSolder, symbol Device:C_Small
- added C16, C17: 10n C0G, Capacitor_SMD:C_0805_2012Metric_Pad1.18x1.45mm_HandSolder, symbol Device:C_Small
- added C20, C21: 10u NICHICON 25V, Capacitor_THT:CP_Radial_D5.0mm_P2.00mm, symbol Device:C_Small
- added J5: Conn_01x03_Pin, Connector_JST:JST_PH_B3B-PH-K_1x03_P2.00mm_Vertical, symbol Connector:Conn_01x03_Pin
- added R8, R9: 100R, Resistor_SMD:R_0805_2012Metric_Pad1.20x1.40mm_HandSolder, symbol Device:R_Small
- added U1: ASDMB-xxxMHz, Oscillator:Oscillator_SMD_Abracon_ASE-4Pin_3.2x2.5mm, symbol Oscillator:ASDMB-xxxMHz
- renumbered C9 to C10, C10 to C11, C13 to C12, C14 to C13, C15 to C14, C16 to C15, C17 to C19, C1 to C2, C19 to C22, C20 to C23, C2 to C3, C3 to C4, C4 to C5, C5 to C6, C6 to C7, C7 to C8, C8 to C9, J5 to J6, R9 to R10, R8 to R11, U1 to U2, U2 to U3
Connections:
- net 3V3: now also C1.1, U1.1 (Standby), U1.4 (VDD)
- net AGND: now also C16.1, C17.2, J5.2 (Pin_2); no longer U3.1 (VINL2), U3.2 (VINR2)
- net GND: now also C1.2, U1.2 (GND)
- net SCLKI: now reaches U3.15 (SCLKI)
- net SCLKI: now also U1.3 (Out)
- net XI: no longer names the net of U3.10 (XI)
- net XO: no longer names the net of U3.9 (XO)
- new net: C16.2, R8.2, U3.1 (VINL2)
- new net: C20.2, R8.1
- new net: C21.2, R9.1
- new net: C17.1, R9.2, U3.2 (VINR2)
- new net MIC_LEFT_IN: C20.1, J5.1 (Pin_1)
- new net MIC_RIGHT_IN: C21.1, J5.3 (Pin_3)
Other:
- moved on the sheet: C18, C19, C22, C23, R10, R11, R4, R5, R6, R7, U3
