File: pcbs/DAC/1.0/DAC.kicad_sch (KiCad schematic)
At the start: 67 parts, among them J1 Conn_01x03_Pin, J11 Conn_01x03_Pin, J2 Conn_01x03_Pin, J3 Conn_01x03_Pin, J4 Conn_01x02_Pin, J5 Conn_01x03_Pin, J6 Conn_01x02_Pin, J7 Conn_01x04_Pin, J8 Conn_01x04_Pin, J9 Conn_01x04_Pin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

Commit message: Updated screenshots
Parts:
- renumbered C32 to C1, C23 to C10, C9 to C11, C33 to C12, C18 to C13, C3 to C14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
