File: pcbs/Extend/1.0/Extend.kicad_pcb (KiCad board)
At the start: 2 copper layers, 85 x 55 mm, 24 parts, among them J1 Conn_01x06_Pin, J10 Conn_01x02_Male, J13 Conn_01x04_Pin, J2 Conn_01x05_Pin, J3 Conn_01x04_Pin, J4 Conn_01x02_Male, J5 Conn_01x02_Male, J6 Conn_01x02_Male, J7 Conn_01x02_Pin, J8 Conn_01x05_Pin, J9 Conn_01x02_Pin, U1 MCP23017_SS

Commit message: Updates
Parts:
- moved R1 6.74 mm to (89.5, 95.4)
- renumbered C3 to C2, C4 to C3, H3 to H2, H2 to H3, J5 to J1, J6 to J10, J9 to J11, J8 to J2, J1 to J4, J4 to J5, J10 to J6, J13 to J7, J2 to J8, J7 to J9, R3 to R1, R4 to R2, R2 to R3, R1 to R4
Routing:
- net RESET: track 42.6 -> 46.3 mm
- net SPDIF_INT1: track 54.7 -> 56.1 mm
- net SDA: track 153.2 -> 154.1 mm
- net CHANSEL4: track 56.0 -> 56.7 mm
- net INTB: track 50.1 -> 49.6 mm
- net SPDIF_INT2: track 55.4 -> 54.9 mm
- net (no net): vias 1 -> 0

Commit message: Updated screenshots
Parts:
- added J12: Conn_01x03_Pin, Connector_JST:JST_PH_B3B-PH-K_1x03_P2.00mm_Vertical, F.Cu at (89.3, 73.5)
- moved J2 10.8 mm to (89.3, 94.5)
- moved R1 10.8 mm to (89.6, 106.2)
- moved J1 10.4 mm to (89.3, 85.0)
Connections:
- net CHANSEL4 renamed CHAN_EN
- U1 pad 24: unconnected-(U1-GPA3-Pad24) -> DAC_XSMT
Routing:
- net GND: track 0.00 -> 168.2 mm, vias 7 -> 10
- net DAC_XSMT: track 0.00 -> 41.8 mm
- net SCL: track 133.4 -> 153.6 mm
- net 3V3: track 81.3 -> 96.1 mm
- net SDA: track 154.1 -> 165.4 mm, vias 1 -> 2
- net ADC_INT: track 39.9 -> 30.1 mm
- net MONOBLOCK_ENABLE: track 33.3 -> 41.6 mm
- net INTA: track 41.4 -> 49.2 mm
- net DSP_EN1: track 30.6 -> 36.0 mm
- net CHAN_EN: track 56.7 -> 61.6 mm
- net INTB: track 49.6 -> 45.0 mm, vias 1 -> 0
- net RESET: track 46.3 -> 50.9 mm
- net DSP_BOOT: track 34.1 -> 37.6 mm
- net CHANSEL1: track 48.4 -> 51.2 mm
- net A2: track 40.0 -> 37.6 mm
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Other:
- board text added: "DAC_CTRL"
