File: pcbs/SPDIF/1.0/spdif.kicad_sch (KiCad schematic)
At the start: 67 parts, among them J1 Conn_01x02_Pin, J10 Conn_01x05_Pin, J11 Conn_01x04_Pin, J12 Conn_01x03_Pin, J13 Conn_01x02_Pin, J2 Conn_01x02_Pin, J3 Conn_01x02_Pin, J4 Conn_01x02_Pin, J5 Conn_01x02_Pin, J6 Conn_01x04_Pin, J7 Conn_01x04_Pin, J8 Conn_01x04_Pin, J9 Conn_01x02_Pin, U1 DA101C_C6931652, U2 DA101C_C6931652, U3 DA101C_C6931652, U4 DA101C_C6931652, U5 74HC7014, U6 DIX9211, U7 AMS1117-3.3, Y1 24.576MHz

Commit message: Updated screenshots
Parts:
- removed C12, C9: 68n C0G, Capacitor_SMD:C_0603_1608Metric, symbol Device:C_Small
- removed R10: 200R, Resistor_SMD:R_0603_1608Metric, symbol Device:R_Small
- removed Y1: 24.576MHz, Crystal:Crystal_SMD_SeikoEpson_FA238-4Pin_3.2x2.5mm, symbol Device:Crystal_GND24_Small
- added C3: 0.1u, Capacitor_SMD:C_0805_2012Metric_Pad1.18x1.45mm_HandSolder, symbol Device:C_Small
- added J3: Conn_01x02_Pin, Connector_JST:JST_XH_B2B-XH-A_1x02_P2.50mm_Vertical, symbol Connector:Conn_01x02_Pin
- added U1: DA101C_C6931652, easyeda2kicad:XFMR-TH_4P-L9.5-W9.0-P5.08-LS10.2_C9900096976, symbol easyeda2kicad:DA101C_C6931652
- added U9: ASDMB-xxxMHz, Oscillator:Oscillator_SMD_Abracon_ASE-4Pin_3.2x2.5mm, symbol Oscillator:ASDMB-xxxMHz
- U2: renamed from U1; Mouser (none) -> 580-DA101C
- U4: renamed from U2; Mouser (none) -> 580-DA101C
- U6: renamed from U3; Mouser (none) -> 580-DA101C
- U8: renamed from U4; Mouser (none) -> 580-DA101C
- renumbered C14 to C10, C8 to C11, C17 to C12, C10 to C13, C11 to C14, C3 to C15, C18 to C16, C5 to C17, C6 to C18, C20 to C2, C4 to C20, C16 to C5, C13 to C6, C15 to C7, C2 to C8, C7 to C9, D2 to D1, D3 to D2, D1 to D3, H3 to H2, H2 to H3, J8 to J1, J5 to J10, J12 to J11, J6 to J12, J7 to J13, J10 to J14, J11 to J2, J1 to J4, J9 to J5, J2 to J6, J13 to J7, J3 to J8, J4 to J9, R12 to R1, R3 to R10, R6 to R11, R8 to R12, R18 to R13, R19 to R14, R7 to R15, R9 to R16, R4 to R17, R16 to R18, R5 to R19, R13 to R2, R14 to R3, R15 to R4, R17 to R5, R1 to R6, R2 to R8, R11 to R9, U7 to U3, U6 to U5, U5 to U7
Connections:
- net 3V3: now also C3.1, U9.1 (Standby), U9.4 (VDD)
- net AGND: now also U1.4; no longer C13.1, C14.1, U5.41 (AGND)
- net GND: now also C3.2, U9.2 (GND)
- net SPDIF_OUT: now also U1.6; no longer U5.6 (MPIO_A3)
- net XTI: now also U9.3 (Out)
- net XTO: no longer names the net of U5.40 (XTO)
- new net FILTGND: C13.1, C14.1, U5.41 (AGND)
- new net SPDIFNEG: J3.1 (Pin_1), U1.3
- new net SPDIFPOS: J3.2 (Pin_2), U1.1
