File: pcbs/dual-psu/1.0/dual-psu.kicad_pcb (KiCad board)
At the start: 2 copper layers, 65 x 95 mm, 97 parts, among them J1 Conn_01x02_Pin, J10 Conn_01x02_Pin, J11 Conn_01x02_Pin, J12 Conn_01x02_Pin, J13 Conn_01x02_Pin, J14 Conn_01x02_Pin, J15 Conn_01x03_Male, J16 Conn_01x03_Male, J17 Conn_01x03_Male, J18 Conn_01x03_Male, J19 Conn_01x03_Male, J2 Conn_01x02_Pin, J20 Conn_01x03_Male, J21 Conn_01x03_Male, J22 Conn_01x03_Pin, J23 Conn_01x03_Male, J24 Conn_01x03_Male, J25 Conn_01x03_Male, J26 Conn_01x03_Male, J27 Conn_01x02_Pin, J28 Conn_01x02_Male, J3 Conn_01x02_Pin, J4 Conn_01x02_Pin, J5 Conn_01x02_Pin, J6 Conn_01x02_Pin, J7 Conn_01x02_Pin, J8 Conn_01x03_Male, J9 Conn_01x03_Male, U1 AMS1117-5.0, U10 INA260, U11 INA260, U12 INA260, U13 TMP100, U14 AP64351SP-13, U2 AMS1117-5.0, U3 INA260, U4 ZLDO1117QG33TA, U5 ZLDO1117QG33TA, U7 LM317_SOT-223, U8 LM337_SOT223, U9 NCP1117-12

Commit message: Updates
Parts:
- C21: renamed from C2; value 16V 470u -> 25V 220u
- moved D5 0.11 mm to (131.0, 37.4)
- moved D6 0.07 mm to (131.0, 39.6)
- renumbered C20 to C1, C15 to C10, C1 to C11, C4 to C12, C10 to C13, C13 to C14, C23 to C15, C26 to C16, C19 to C17, C11 to C18, C14 to C19, C3 to C2, C8 to C20, C18 to C22, C28 to C23, C30 to C24, C6 to C25, C27 to C26, C7 to C27, C31 to C28, C5 to C3, C16 to C30, C9 to C4, C12 to C5, C21 to C6, C24 to C7, C22 to C8, C25 to C9, D6 to D1, D7 to D2, D4 to D3, D3 to D4, D1 to D5, D2 to D6, D5 to D7, H3 to H2, H2 to H3, J3 to J1, J19 to J10, J21 to J11, J4 to J12, J7 to J13, J15 to J14, J24 to J15, J11 to J16, J14 to J17, J28 to J18, J9 to J19, J6 to J2, J25 to J20, J8 to J21, J26 to J22, J1 to J23, J12 to J24, J2 to J25, J27 to J26, J17 to J27, J5 to J28, J16 to J3, J23 to J4, J18 to J5, J20 to J6, J10 to J7, J13 to J8, J22 to J9, R16 to R1, R2 to R10, R6 to R11, R8 to R12, R3 to R13, R7 to R14, R14 to R2, R10 to R3, R12 to R4, R15 to R5, R17 to R6, R4 to R7, R5 to R8, R1 to R9, U13 to U11, U9 to U12, U14 to U13, U4 to U3, U5 to U4, U7 to U5, U8 to U6, U11 to U7, U12 to U8, U3 to U9
Routing:
- net DC_POS: track 97.1 -> 98.1 mm
- net SCL: track 130.4 -> 129.5 mm

Commit message: Updating readmes
Parts:
- added J29: Conn_01x02_Pin, Connector_JST:JST_PH_B2B-PH-K_1x02_P2.00mm_Vertical, F.Cu at (161.7, 44.8)
- D1, D2, D7: footprint LED_SMD:LED_0805_2012Metric_Pad1.15x1.40mm_HandSolder -> LED_SMD:LED_0603_1608Metric
- moved J28 5.00 mm to (161.7, 52.2)
- moved D1 0.29 mm to (122.0, 101.4)
- moved D2 0.27 mm to (122.0, 103.1)
Routing:
- net AGND: track 92.9 -> 87.9 mm
Other:
- board text added: "RELAY_GND"
