File: pcbs/dual-psu/1.0/dual-psu.kicad_sch (KiCad schematic)
At the start: 97 parts, among them J1 Conn_01x02_Pin, J10 Conn_01x02_Pin, J11 Conn_01x02_Pin, J12 Conn_01x02_Pin, J13 Conn_01x02_Pin, J14 Conn_01x02_Pin, J15 Conn_01x03_Male, J16 Conn_01x03_Male, J17 Conn_01x03_Male, J18 Conn_01x03_Male, J19 Conn_01x03_Male, J2 Conn_01x02_Pin, J20 Conn_01x03_Male, J21 Conn_01x03_Male, J22 Conn_01x03_Pin, J23 Conn_01x03_Male, J24 Conn_01x03_Male, J25 Conn_01x03_Male, J26 Conn_01x03_Male, J27 Conn_01x02_Pin, J28 Conn_01x02_Male, J3 Conn_01x02_Pin, J4 Conn_01x02_Pin, J5 Conn_01x02_Pin, J6 Conn_01x02_Pin, J7 Conn_01x02_Pin, J8 Conn_01x03_Male, J9 Conn_01x03_Male, U1 AMS1117-5.0, U10 INA260, U11 INA260, U12 INA260, U13 TMP100, U14 AP64351SP-13, U2 AMS1117-5.0, U3 INA260, U4 ZLDO1117QG33TA, U5 ZLDO1117QG33TA, U7 LM317_SOT-223, U8 LM337_SOT223, U9 NCP1117-12

Commit message: Updates
Parts:
- C21: renamed from C2; value 16V 470u -> 25V 220u
- renumbered C20 to C1, C15 to C10, C1 to C11, C4 to C12, C10 to C13, C13 to C14, C23 to C15, C26 to C16, C19 to C17, C11 to C18, C14 to C19, C3 to C2, C8 to C20, C18 to C22, C28 to C23, C30 to C24, C6 to C25, C27 to C26, C7 to C27, C31 to C28, C5 to C3, C16 to C30, C9 to C4, C12 to C5, C21 to C6, C24 to C7, C22 to C8, C25 to C9, D6 to D1, D7 to D2, D4 to D3, D3 to D4, D1 to D5, D2 to D6, D5 to D7, H3 to H2, H2 to H3, J3 to J1, J19 to J10, J21 to J11, J4 to J12, J7 to J13, J15 to J14, J24 to J15, J11 to J16, J14 to J17, J28 to J18, J9 to J19, J6 to J2, J25 to J20, J8 to J21, J26 to J22, J1 to J23, J12 to J24, J2 to J25, J27 to J26, J17 to J27, J5 to J28, J16 to J3, J23 to J4, J18 to J5, J20 to J6, J10 to J7, J13 to J8, J22 to J9, R16 to R1, R2 to R10, R6 to R11, R8 to R12, R3 to R13, R7 to R14, R14 to R2, R10 to R3, R12 to R4, R15 to R5, R17 to R6, R4 to R7, R5 to R8, R1 to R9, U13 to U11, U9 to U12, U14 to U13, U4 to U3, U5 to U4, U7 to U5, U8 to U6, U11 to U7, U12 to U8, U3 to U9
Other:
- moved on the sheet: C10, C13, C14, C24, C28, D3, D4, D5, D6, J23, J25, L1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

Commit message: Updating readmes
Parts:
- added J29: Conn_01x02_Pin, Connector_JST:JST_PH_B2B-PH-K_1x02_P2.00mm_Vertical, symbol Connector:Conn_01x02_Pin
- D1, D2, D7: footprint LED_SMD:LED_0805_2012Metric_Pad1.15x1.40mm_HandSolder -> LED_SMD:LED_0603_1608Metric
Connections:
- net RELAYGND: now also J29.1 (Pin_1), J29.2 (Pin_2)
Changed lines of the file:
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@@
 		)
 	)
+	(global_label "RELAYGND"
+		(shape input)
+		(at 262.89 44.45 0)
+		(fields_autoplaced yes)
+		(effects
+			(font
+				(size 1.27 1.27)
+			)
+			(justify left)
+		)
+		(property "Intersheetrefs" "${INTERSHEET_REFS}"
+			(at 275.37 44.45 0)
+			(effects
+				(font
+					(size 1.27 1.27)
+				)
+				(justify left)
+				(hide yes)
+			)
+		)
+	)
 	(global_label "3V3_1"
 		(shape input)
@@
 		)
 	)
+	(global_label "RELAYGND"
+		(shape input)
+		(at 262.89 41.91 0)
+		(fields_autoplaced yes)
+		(effects
+			(font
+				(size 1.27 1.27)
+			)
+			(justify left)
+		)
+		(property "Intersheetrefs" "${INTERSHEET_REFS}"
+			(at 275.37 41.91 0)
+			(effects
+				(font
+					(size 1.27 1.27)
+				)
+				(justify left)
+				(hide yes)
+			)
+		)
+	)
 	(global_label "3V3_1"
 		(shape input)
@@
 			)
 		)
-		(property "Footprint" "LED_SMD:LED_0805_2012Metric_Pad1.15x1.40mm_HandSolder"
+		(property "Footprint" "LED_SMD:LED_0603_1608Metric"
 			(at 367.919 44.323 0)
 			(effects
@@
 	)
 	(symbol
+		(lib_id "Connector:Conn_01x02_Pin")
+		(at 257.81 41.91 0)
+		(unit 1)
+		(exclude_from_sim no)
+		(in_bom yes)
+		(on_board yes)
+		(dnp no)
+		(fields_autoplaced yes)
+		(property "Reference" "J29"
+			(at 258.445 36.322 0)
+			(effects
+				(font
+					(size 1.27 1.27)
+				)
+			)
+		)
+		(property "Value" "Conn_01x02_Pin"
+			(at 258.445 38.862 0)
+			(effects
+				(font
+					(size 1.27 1.27)
+				)
+			)
+		)
+		(property "Footprint" "Connector_JST:JST_PH_B2B-PH-K_1x02_P2.00mm_Vertical"
+			(at 257.81 41.91 0)
+			(effects
+				(font
+					(size 1.27 1.27)
+				)
+				(hide yes)
+			)
+		)
+		(property "Datasheet" "~"
+			(at 257.81 41.91 0)
+			(effects
+				(font
+					(size 1.27 1.27)
+				)
+				(hide yes)
+			)
+		)
+		(property "Description" ""
+			(at 257.81 41.91 0)
+			(effects
+				(font
+					(size 1.27 1.27)
+				)
+				(hide yes)
+			)
+		)
+		(pin "1"
+		)
+		(pin "2"
+		)
+		(instances
+			(project "dual-psu"
+				(path "/5486715c-d46c-4c73-9a76-76411783f9bd"
+					(reference "J29")
+					(unit 1)
+				)
+			)
+		)
+	)
+	(symbol
 		(lib_id "Device:C_Polarized_Small")
 		(at 162.56 147.32 0)
@@
 			)
 		)
-		(property "Footprint" "LED_SMD:LED_0805_2012Metric_Pad1.15x1.40mm_HandSolder"
+		(property "Footprint" "LED_SMD:LED_0603_1608Metric"
 			(at 382.27 46.99 0)
 			(effects
@@
 			)
 		)
-		(property "Footprint" "LED_SMD:LED_0805_2012Metric_Pad1.15x1.40mm_HandSolder"
+		(property "Footprint" "LED_SMD:LED_0603_1608Metric"
 			(at 354.33 46.99 0)
 			(effects

Commit message: Updates to pcbs
Parts:
- R13: value 170K -> 180K; Mouser (none) -> 603-RC0603JR-10180KL
- U13: Mouser (none) -> 621-AP64351SP-13
Changed lines of the file:
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@@
 			)
 		)
-		(property "Value" "170K"
+		(property "Value" "180K"
 			(at 373.126 121.9199 0)
 			(effects
@@
 			)
 		)
+		(property "Mouser" " 603-RC0603JR-10180KL "
+			(at 370.84 120.65 0)
+			(effects
+				(font
+					(size 1.27 1.27)
+				)
+				(hide yes)
+			)
+		)
 		(pin "1"
 		)
@@
 			(effects
 				(font
+					(size 1.27 1.27)
+				)
+				(hide yes)
+			)
+		)
+		(property "Mouser" " 621-AP64351SP-13 "
+			(at 337.82 119.38 0)
+			(effects
+				(font
