File: pcbs/_ready/lm3886/1.0/lm3886.kicad_sch (KiCad schematic)
At the start: 43 parts, among them J1 Conn_01x02_Male, J11 Conn_01x03_Male, J12 Conn_01x02_Male, J2 Conn_01x02_Male, J3 Conn_01x03_Male, J4 Conn_01x02_Male, J5 Conn_01x02_Male, J6 Conn_01x02_Male, J7 Conn_01x03_Male, J8 Conn_01x02_Male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

Commit message: Updates to pcbs
Parts:
- C3, C4: value 22U 50V -> 47U 50V
- R2: value 750R -> 1.4k
Changed lines of the file:
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@@
 			)
 		)
-		(property "Value" "750R"
+		(property "Value" "1.4k"
 			(at 92.71 173.9899 0)
 			(effects
@@
 			)
 		)
-		(property "Value" "22U 50V"
+		(property "Value" "47U 50V"
 			(at 99.7839 80.01 90)
 			(effects
@@
 			)
 		)
-		(property "Value" "22U 50V"
+		(property "Value" "47U 50V"
 			(at 100.8761 129.54 90)
 			(effects
