File: pcbs/_ready/lm3886/1.0/lm3886.kicad_pcb (KiCad board)
At the start: 4 copper layers, 55 x 95 mm, 43 parts, among them J1 Conn_01x02_Male, J11 Conn_01x03_Male, J12 Conn_01x02_Male, J2 Conn_01x02_Male, J3 Conn_01x03_Male, J4 Conn_01x02_Male, J5 Conn_01x02_Male, J6 Conn_01x02_Male, J7 Conn_01x03_Male, J8 Conn_01x02_Male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

Commit message: More work on PCBs
Parts:
- C3, C4: value 22U 50V -> 47U 50V
- R2: value 750R -> 1.4k
Changed lines of the file:
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@@
 		(property ki_fp_filters "C_*")
 		(sheetname "Root")
-		(sheetfile "LM3886.kicad_sch")
+		(sheetfile "lm3886.kicad_sch")
 		(attr smd)
 		(fp_line
@@
 			)
 		)
-		(property "Value" "750R"
+		(property "Value" "1.4k"
 			(at 0 1.82 90)
 			(layer "F.Fab")
@@
 		(property ki_fp_filters "R_*")
 		(sheetname "Root")
-		(sheetfile "LM3886.kicad_sch")
+		(sheetfile "lm3886.kicad_sch")
 		(attr smd)
 		(fp_line
@@
 		(property ki_fp_filters "Connector*:*_1x??_*")
 		(sheetname "Root")
-		(sheetfile "LM3886.kicad_sch")
+		(sheetfile "lm3886.kicad_sch")
 		(attr through_hole)
 		(fp_line
@@
 		(property ki_fp_filters "Connector*:*_1x??_*")
 		(sheetname "Root")
-		(sheetfile "LM3886.kicad_sch")
+		(sheetfile "lm3886.kicad_sch")
 		(attr through_hole)
 		(fp_line
@@
 			)
 		)
-		(property "Value" "22U 50V"
+		(property "Value" "47U 50V"
 			(at 1.25 4.4 180)
 			(unlocked yes)
@@
 		(property ki_fp_filters "CP_*")
 		(sheetname "Root")
-		(sheetfile "LM3886.kicad_sch")
+		(sheetfile "lm3886.kicad_sch")
 		(attr through_hole)
 		(fp_line
@@
 		(property ki_fp_filters "R_*")
 		(sheetname "Root")
-		(sheetfile "LM3886.kicad_sch")
+		(sheetfile "lm3886.kicad_sch")
 		(attr smd)
 		(fp_line
@@
 		(property ki_fp_filters "R_*")
 		(sheetname "Root")
-		(sheetfile "LM3886.kicad_sch")
+		(sheetfile "lm3886.kicad_sch")
 		(attr smd)
 		(fp_line
@@
 			)
 		)
-		(property "Value" "22U 50V"
+		(property "Value" "47U 50V"
 			(at 1.25 4.4 0)
 			(unlocked yes)
@@
 		(property ki_fp_filters "CP_*")
 		(sheetname "Root")
-		(sheetfile "LM3886.kicad_sch")
+		(sheetfile "lm3886.kicad_sch")
 		(attr through_hole)
 		(fp_line
@@
 		(property ki_fp_filters "CP_*")
 		(sheetname "Root")
-		(sheetfile "LM3886.kicad_sch")
+		(sheetfile "lm3886.kicad_sch")
 		(attr through_hole)
 		(fp_line
@@
 		(property ki_fp_filters "MountingHole*")
 		(sheetname "Root")
-		(sheetfile "LM3886.kicad_sch")
+		(sheetfile "lm3886.kicad_sch")
 		(attr through_hole)
 		(fp_text user "${REFERENCE}"
@@
 		(property ki_fp_filters "CP_*")
 		(sheetname "Root")
-		(sheetfile "LM3886.kicad_sch")
+		(sheetfile "lm3886.kicad_sch")
 		(attr smd)
 		(fp_line
@@
 		(property ki_fp_filters "R_*")
 		(sheetname "Root")
-		(sheetfile "LM3886.kicad_sch")
+		(sheetfile "lm3886.kicad_sch")
 		(attr smd)
 		(fp_line
@@
 		(property ki_fp_filters "Connector*:*_1x??_*")
 		(sheetname "Root")
-		(sheetfile "LM3886.kicad_sch")
+		(sheetfile "lm3886.kicad_sch")
 		(attr through_hole)
 		(fp_line
@@
 		(property ki_fp_filters "Connector*:*_1x??_*")
 		(sheetname "Root")
-		(sheetfile "LM3886.kicad_sch")
+		(sheetfile "lm3886.kicad_sch")
 		(attr through_hole)
 		(fp_line
@@
 		(property ki_fp_filters "R_*")
 		(sheetname "Root")
-		(sheetfile "LM3886.kicad_sch")
+		(sheetfile "lm3886.kicad_sch")
 		(attr smd)
 		(fp_line
@@
 		(property ki_fp_filters "Connector*:*_1x??_*")
 		(sheetname "Root")
-		(sheetfile "LM3886.kicad_sch")
+		(sheetfile "lm3886.kicad_sch")
 		(attr through_hole)
 		(fp_line
@@
 		(property ki_fp_filters "CP_*")
 		(sheetname "Root")
-		(sheetfile "LM3886.kicad_sch")
+		(sheetfile "lm3886.kicad_sch")
 		(attr smd)
 		(fp_line
@@
 		(property ki_fp_filters "R_*")
 		(sheetname "Root")
-		(sheetfile "LM3886.kicad_sch")
+		(sheetfile "lm3886.kicad_sch")
 		(attr smd)
 		(fp_line
@@
 		(property ki_fp_filters "MountingHole*")
 		(sheetname "Root")
-		(sheetfile "LM3886.kicad_sch")
+		(sheetfile "lm3886.kicad_sch")
 		(attr through_hole)
 		(fp_text user "${REFERENCE}"
@@
 		(property ki_fp_filters "C_*")
 		(sheetname "Root")
-		(sheetfile "LM3886.kicad_sch")
+		(sheetfile "lm3886.kicad_sch")
 		(attr smd)
 		(fp_line
@@
 		(property ki_fp_filters "TO?220*StaggerOdd*")
 		(sheetname "Root")
-		(sheetfile "LM3886.kicad_sch")
+		(sheetfile "lm3886.kicad_sch")
 		(attr through_hole)
 		(fp_line
@@
 		(property ki_fp_filters "C_*")
 		(sheetname "Root")
-		(sheetfile "LM3886.kicad_sch")
+		(sheetfile "lm3886.kicad_sch")
 		(attr through_hole)
 		(fp_circle
@@
 		(property ki_fp_filters "Connector*:*_1x??_*")
 		(sheetname "Root")
-		(sheetfile "LM3886.kicad_sch")
+		(sheetfile "lm3886.kicad_sch")
 		(attr through_hole)
 		(fp_line
@@
 		(property ki_fp_filters "C_*")
 		(sheetname "Root")
-		(sheetfile "LM3886.kicad_sch")
+		(sheetfile "lm3886.kicad_sch")
 		(attr through_hole)
 		(fp_line
@@
 		(property ki_fp_filters "R_*")
 		(sheetname "Root")
-		(sheetfile "LM3886.kicad_sch")
+		(sheetfile "lm3886.kicad_sch")
 		(attr smd)
 		(fp_line
@@
 		(property ki_fp_filters "MountingHole*")
 		(sheetname "Root")
-		(sheetfile "LM3886.kicad_sch")
+		(sheetfile "lm3886.kicad_sch")
 		(attr through_hole)
 		(fp_text user "${REFERENCE}"
@@
 		(property ki_fp_filters "R_*")
 		(sheetname "Root")
-		(sheetfile "LM3886.kicad_sch")
+		(sheetfile "lm3886.kicad_sch")
 		(attr smd)
 		(fp_line
@@
 		(property ki_fp_filters "Connector*:*_1x??_*")
 		(sheetname "Root")
-		(sheetfile "LM3886.kicad_sch")
+		(sheetfile "lm3886.kicad_sch")
 		(attr through_hole)
 		(fp_line
@@
 		(property ki_fp_filters "Connector*:*_1x??_*")
 		(sheetname "Root")
-		(sheetfile "LM3886.kicad_sch")
+		(sheetfile "lm3886.kicad_sch")
 		(attr through_hole)
 		(fp_line
@@
 		(property ki_fp_filters "Connector*:*_1x??_*")
 		(sheetname "Root")
-		(sheetfile "LM3886.kicad_sch")
+		(sheetfile "lm3886.kicad_sch")
 		(attr through_hole)
 		(fp_line
@@
 		(property ki_fp_filters "LED* LED_SMD:* LED_THT:*")
 		(sheetname "Root")
-		(sheetfile "LM3886.kicad_sch")
+		(sheetfile "lm3886.kicad_sch")
 		(attr smd)
 		(fp_line
@@
 		(property ki_fp_filters "R_*")
 		(sheetname "Root")
-		(sheetfile "LM3886.kicad_sch")
+		(sheetfile "lm3886.kicad_sch")
 		(attr smd)
 		(fp_line
@@
 		(property ki_fp_filters "CP_*")
 		(sheetname "Root")
-		(sheetfile "LM3886.kicad_sch")
+		(sheetfile "lm3886.kicad_sch")
 		(attr through_hole)
 		(fp_line
@@
 		(property ki_fp_filters "C_*")
 		(sheetname "Root")
-		(sheetfile "LM3886.kicad_sch")
+		(sheetfile "lm3886.kicad_sch")
 		(attr smd)
 		(fp_line
@@
 		(property ki_fp_filters "CP_*")
 		(sheetname "Root")
-		(sheetfile "LM3886.kicad_sch")
+		(sheetfile "lm3886.kicad_sch")
 		(attr through_hole)
 		(fp_line
@@
 		(property ki_fp_filters "MountingHole*")
 		(sheetname "Root")
-		(sheetfile "LM3886.kicad_sch")
+		(sheetfile "lm3886.kicad_sch")
 		(attr through_hole)
 		(fp_text user "${REFERENCE}"
@@
 		(property ki_fp_filters "R_*")
 		(sheetname "Root")
-		(sheetfile "LM3886.kicad_sch")
+		(sheetfile "lm3886.kicad_sch")
 		(attr smd)
 		(fp_line
@@
 		(property ki_fp_filters "R_*")
 		(sheetname "Root")
-		(sheetfile "LM3886.kicad_sch")
+		(sheetfile "lm3886.kicad_sch")
 		(attr smd)
 		(fp_line
@@
 		(property ki_fp_filters "Connector*:*_1x??_*")
 		(sheetname "Root")
-		(sheetfile "LM3886.kicad_sch")
+		(sheetfile "lm3886.kicad_sch")
 		(attr through_hole)
 		(fp_line
@@
 		(property ki_fp_filters "Choke_* *Coil* Inductor_* L_*")
 		(sheetname "Root")
-		(sheetfile "LM3886.kicad_sch")
+		(sheetfile "lm3886.kicad_sch")
 		(attr through_hole)
 		(fp_circle
@@
 		(property ki_fp_filters "LED* LED_SMD:* LED_THT:*")
 		(sheetname "Root")
-		(sheetfile "LM3886.kicad_sch")
+		(sheetfile "lm3886.kicad_sch")
 		(attr smd)
 		(fp_line
@@
 		(property ki_fp_filters "CP_*")
 		(sheetname "Root")
-		(sheetfile "LM3886.kicad_sch")
+		(sheetfile "lm3886.kicad_sch")
 		(attr through_hole)
 		(fp_line
@@
 		(property ki_fp_filters "Connector*:*_1x??_*")
 		(sheetname "Root")
-		(sheetfile "LM3886.kicad_sch")
+		(sheetfile "lm3886.kicad_sch")
 		(attr through_hole)
 		(fp_line
@@
 		)
 	)
+	(gr_rect
+		(start 77.2 43.65)
+		(end 82.2 48.65)
+		(stroke
+			(width 0.1)
+			(type solid)
+		)
+		(fill solid)
+		(layer "F.SilkS")
+	)
 	(gr_line
