File: pcbs/_ready/vinyl/1.0/vinyl.kicad_sch (KiCad schematic)
At the start: 59 parts, among them J1 Conn_01x03_Male, J2 Conn_01x03_Male, J3 Conn_01x03_Pin, J4 Conn_01x03_Male, J5 Conn_01x03_Male, J6 Conn_01x03_Male, U1 OPA2134, U2 OPA2134

Commit message: Updates to pcbs
Parts:
- C2, C9: Mouser (none) -> 81-GRM3195C1H104GA5D
- R1, R10: Mouser (none) -> 603-RT0805FRE072K2L
- R11, R2: Mouser (none) -> 603-RT0805FRE0747KL
- R12, R3: Mouser (none) -> 603-RT0805FRE074K7L
- R13, R17, R4, R8: Mouser (none) -> 603-RT0805FRE10100KL
- R14, R5: Mouser (none) -> 603-RT0805FRE07750RL
- R15, R6: Mouser (none) -> 603-RT0805FRE072K7L
- R16, R7: Mouser (none) -> 603-RT0805FRE1310KL
- R18, R9: Mouser (none) -> 603-RT0805FRE07180KL
- U1, U2: value OPA2134 -> OPA1656; Mouser (none) -> 595-OPA1656IDR
Changed lines of the file:
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@@
 			)
 		)
+		(property "Mouser" " 603-RT0805FRE072K7L "
+			(at 203.835 97.663 0)
+			(effects
+				(font
+					(size 1.27 1.27)
+				)
+				(hide yes)
+			)
+		)
 		(pin "1"
 		)
@@
 			)
 		)
+		(property "Mouser" " 603-RT0805FRE0747KL "
+			(at 140.97 82.677 0)
+			(effects
+				(font
+					(size 1.27 1.27)
+				)
+				(hide yes)
+			)
+		)
 		(pin "1"
 		)
@@
 			)
 		)
+		(property "Mouser" " 603-RT0805FRE072K2L "
+			(at 41.021 80.01 90)
+			(effects
+				(font
+					(size 1.27 1.27)
+				)
+				(hide yes)
+			)
+		)
 		(pin "1"
 		)
@@
 			)
 		)
+		(property "Mouser" " 603-RT0805FRE0747KL "
+			(at 36.322 83.947 0)
+			(effects
+				(font
+					(size 1.27 1.27)
+				)
+				(hide yes)
+			)
+		)
 		(pin "1"
 		)
@@
 			)
 		)
+		(property "Mouser" " 603-RT0805FRE074K7L "
+			(at 44.45 92.583 0)
+			(effects
+				(font
+					(size 1.27 1.27)
+				)
+				(hide yes)
+			)
+		)
 		(pin "1"
 		)
@@
 			)
 		)
+		(property "Mouser" " 603-RT0805FRE1310KL "
+			(at 106.68 74.93 0)
+			(effects
+				(font
+					(size 1.27 1.27)
+				)
+				(hide yes)
+			)
+		)
 		(pin "1"
 		)
@@
 			)
 		)
+		(property "Mouser" " 603-RT0805FRE07180KL "
+			(at 203.073 77.47 0)
+			(effects
+				(font
+					(size 1.27 1.27)
+				)
+				(hide yes)
+			)
+		)
 		(pin "1"
 		)
@@
 			)
 		)
+		(property "Mouser" " 603-RT0805FRE10100KL "
+			(at 94.869 95.758 90)
+			(effects
+				(font
+					(size 1.27 1.27)
+				)
+				(hide yes)
+			)
+		)
 		(pin "1"
 		)
@@
 			)
 		)
+		(property "Mouser" " 81-GRM3195C1H104GA5D "
+			(at 170.307 97.028 0)
+			(effects
+				(font
+					(size 1.27 1.27)
+				)
+				(hide yes)
+			)
+		)
 		(pin "1"
 		)
@@
 			)
 		)
+		(property "Mouser" " 603-RT0805FRE072K2L "
+			(at 145.669 78.74 90)
+			(effects
+				(font
+					(size 1.27 1.27)
+				)
+				(hide yes)
+			)
+		)
 		(pin "1"
 		)
@@
 			)
 		)
+		(property "Mouser" " 603-RT0805FRE072K7L "
+			(at 99.187 99.822 0)
+			(effects
+				(font
+					(size 1.27 1.27)
+				)
+				(hide yes)
+			)
+		)
 		(pin "1"
 		)
@@
 			)
 		)
+		(property "Mouser" " 603-RT0805FRE10100KL "
+			(at 161.29 97.028 0)
+			(effects
+				(font
+					(size 1.27 1.27)
+				)
+				(hide yes)
+			)
+		)
 		(pin "1"
 		)
@@
 			)
 		)
-		(property "Value" "OPA2134"
+		(property "Value" "OPA1656"
 			(at 189.23 64.516 0)
 			(effects
@@
 			)
 		)
+		(property "Mouser" "595-OPA1656IDR"
+			(at 189.23 90.17 0)
+			(effects
+				(font
+					(size 1.27 1.27)
+				)
+				(hide yes)
+			)
+		)
 		(pin "1"
 		)
@@
 			)
 		)
+		(property "Mouser" " 603-RT0805FRE07750RL "
+			(at 69.088 95.758 90)
+			(effects
+				(font
+					(size 1.27 1.27)
+				)
+				(hide yes)
+			)
+		)
 		(pin "1"
 		)
@@
 			)
 		)
+		(property "Mouser" " 603-RT0805FRE074K7L "
+			(at 149.098 91.313 0)
+			(effects
+				(font
+					(size 1.27 1.27)
+				)
+				(hide yes)
+			)
+		)
 		(pin "1"
 		)
@@
 			)
 		)
+		(property "Mouser" " 603-RT0805FRE07180KL "
+			(at 99.06 74.93 0)
+			(effects
+				(font
+					(size 1.27 1.27)
+				)
+				(hide yes)
+			)
+		)
 		(pin "1"
 		)
@@
 			)
 		)
+		(property "Mouser" " 603-RT0805FRE10100KL "
+			(at 56.642 98.298 0)
+			(effects
+				(font
+					(size 1.27 1.27)
+				)
+				(hide yes)
+			)
+		)
 		(pin "1"
 		)
@@
 			)
 		)
+		(property "Mouser" " 603-RT0805FRE1310KL "
+			(at 209.296 74.041 0)
+			(effects
+				(font
+					(size 1.27 1.27)
+				)
+				(hide yes)
+			)
+		)
 		(pin "1"
 		)
@@
 			)
 		)
+		(property "Mouser" " 81-GRM3195C1H104GA5D "
+			(at 65.659 98.298 0)
+			(effects
+				(font
+					(size 1.27 1.27)
+				)
+				(hide yes)
+			)
+		)
 		(pin "1"
 		)
@@
 			)
 		)
+		(property "Mouser" " 603-RT0805FRE07750RL "
+			(at 173.736 94.488 90)
+			(effects
+				(font
+					(size 1.27 1.27)
+				)
+				(hide yes)
+			)
+		)
 		(pin "1"
 		)
@@
 			)
 		)
+		(property "Mouser" " 603-RT0805FRE10100KL "
+			(at 199.517 94.488 90)
+			(effects
+				(font
+					(size 1.27 1.27)
+				)
+				(hide yes)
+			)
+		)
 		(pin "1"
 		)
@@
 			)
 		)
-		(property "Value" "OPA2134"
+		(property "Value" "OPA1656"
 			(at 84.582 65.786 0)
 			(effects
@@
 			(at 84.582 91.44 0)
 			(effects
+				(font
+					(size 1.27 1.27)
+				)
+				(hide yes)
+			)
+		)
+		(property "Mouser" "595-OPA1656IDR"
+			(at 84.582 91.44 0)
+			(effects
