File: pcbs/_ready/vinyl/1.0/vinyl.kicad_pcb (KiCad board)
At the start: 2 copper layers, 85 x 55 mm, 59 parts, among them J1 Conn_01x03_Male, J2 Conn_01x03_Male, J3 Conn_01x03_Pin, J4 Conn_01x03_Male, J5 Conn_01x03_Male, J6 Conn_01x03_Male, U1 OPA2134, U2 OPA2134

Commit message: More work on PCBs
Routing:
- net V-: track 179.8 -> 180.4 mm
- net AGND: vias 3 -> 5
Changed lines of the file:
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@@
 		)
+	)
+	(gr_rect
+		(start 132.1 87.2)
+		(end 137.1 92.2)
+		(stroke
+			(width 0.1)
+			(type solid)
+		)
+		(fill solid)
+		(layer "F.SilkS")
 	)
 	(gr_line
@@
 	)
 	(segment
-		(start 214.1387 114.3387)
-		(end 213.4 113.6)
+		(start 214.9 123.6)
+		(end 214.9 115.1)
 		(width 0.3)
 		(layer "B.Cu")
@@
 	)
 	(segment
-		(start 214.1387 124.3613)
-		(end 214.1387 114.3387)
-		(width 0.3)
-		(layer "B.Cu")
-		(net 1)
-	)
-	(segment
 		(start 134 125.6)
 		(end 132.6471 124.2471)
@@
 	)
 	(segment
+		(start 212.9 125.6)
+		(end 214.9 123.6)
+		(width 0.3)
+		(layer "B.Cu")
+		(net 1)
+	)
+	(segment
 		(start 163.3242 89.6624)
 		(end 164.55 88.4366)
@@
 	)
 	(segment
-		(start 212.9 125.6)
-		(end 214.1387 124.3613)
-		(width 0.3)
-		(layer "B.Cu")
-		(net 1)
-	)
-	(segment
 		(start 154.1 111.1)
 		(end 136.3 111.1)
@@
 	)
 	(segment
+		(start 214.9 115.1)
+		(end 213.4 113.6)
+		(width 0.3)
+		(layer "B.Cu")
+		(net 1)
+	)
+	(segment
 		(start 132.6471 124.2471)
 		(end 132.6471 111.0049)
@@
 	)
 	(via
-		(at 185.4 95.1)
+		(at 213.6 117.9)
 		(size 0.6)
 		(drill 0.3)
@@
 		(net 7)
 	)
-	(segment
-		(start 156.0643 92.2124)
+	(via
+		(at 185.4 95.1)
+		(size 0.6)
+		(drill 0.3)
+		(layers "F.Cu" "B.Cu")
+		(free yes)
+		(net 7)
+	)
+	(via
+		(at 169.4 112)
+		(size 0.6)
+		(drill 0.3)
+		(layers "F.Cu" "B.Cu")
+		(free yes)
+		(net 7)
+	)
+	(segment
+		(start 160.4576 91.1)
+		(end 154.9519 91.1)
+		(width 0.3)
+		(layer "F.Cu")
+		(net 9)
+	)
+	(segment
+		(start 154.9519 91.1)
 		(end 151.9254 88.0735)
 		(width 0.3)
@@
 	(segment
 		(start 161.57 92.2124)
-		(end 156.0643 92.2124)
-		(width 0.3)
-		(layer "F.Cu")
+		(end 160.4576 91.1)
+		(width 0.3)
+		(layer "F.Cu")
