File: pcbs/dac/1.0/dac.kicad_pcb (KiCad board)
At the start: 2 copper layers, 85 x 55 mm, 67 parts, among them J1 Conn_01x04_Pin, J10 Conn_01x02_Pin, J2 Conn_01x03_Pin, J3 Conn_01x04_Pin, J4 Conn_01x03_Pin, J5 Conn_01x04_Pin, J6 Conn_01x03_Pin, J7 Conn_01x02_Pin, J8 Conn_01x03_Pin, J9 Conn_01x03_Pin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

Commit message: Updates to pcbs
Parts:
- removed U4: DA101C_C6931652, easyeda2kicad:XFMR-TH_4P-L9.5-W9.0-P5.08-LS10.2_C9900096976
- added U6: DA101C_C6931652, easyeda2kicad:XFMR-TH_4P-L9.5-W9.0-P5.08-LS10.2_C9900096976, F.Cu at (128.7, 64.4)
- U5: value AMS1117-3.3 -> ZLDO1117QG33TA
