File: pcbs/dac/1.0/dac.kicad_sch (KiCad schematic)
At the start: 67 parts, among them J1 Conn_01x04_Pin, J10 Conn_01x02_Pin, J2 Conn_01x03_Pin, J3 Conn_01x04_Pin, J4 Conn_01x03_Pin, J5 Conn_01x04_Pin, J6 Conn_01x03_Pin, J7 Conn_01x02_Pin, J8 Conn_01x03_Pin, J9 Conn_01x03_Pin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

Commit message: Updates to pcbs
Parts:
- removed U4: DA101C_C6931652, easyeda2kicad:XFMR-TH_4P-L9.5-W9.0-P5.08-LS10.2_C9900096976, symbol easyeda2kicad:DA101C_C6931652
- added U6: DA101C_C6931652, easyeda2kicad:XFMR-TH_4P-L9.5-W9.0-P5.08-LS10.2_C9900096976, symbol easyeda2kicad:DA101C_C6931652
- C16, C18, C27, C30, C4, C7: Mouser (none) -> 603-CC1206JKX78BB225
- U1, U2, U3: Mouser 595-PCM5142PWR -> 595-PCM5122PWR
- U5: value AMS1117-3.3 -> ZLDO1117QG33TA
Connections:
- net AGND: now also U6.3
- net SUBWOOFER: now also U6.1
- net SW_NEG: now also U6.4
- net SW_OUT: now also U6.6
Changed lines of the file:
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@@
 	)
 	(symbol
-		(lib_id "easyeda2kicad:DA101C_C6931652")
-		(at 220.98 41.91 0)
-		(unit 1)
-		(exclude_from_sim no)
-		(in_bom yes)
-		(on_board yes)
-		(dnp no)
-		(fields_autoplaced yes)
-		(property "Reference" "U4"
-			(at 220.9846 31.75 0)
-			(effects
-				(font
-					(size 1.27 1.27)
-				)
-			)
-		)
-		(property "Value" "DA101C_C6931652"
-			(at 220.9846 34.29 0)
-			(effects
-				(font
-					(size 1.27 1.27)
-				)
-			)
-		)
-		(property "Footprint" "easyeda2kicad:XFMR-TH_4P-L9.5-W9.0-P5.08-LS10.2_C9900096976"
-			(at 220.98 54.61 0)
-			(effects
-				(font
-					(size 1.27 1.27)
-				)
-				(hide yes)
-			)
-		)
-		(property "Datasheet" ""
-			(at 220.98 41.91 0)
-			(effects
-				(font
-					(size 1.27 1.27)
-				)
-				(hide yes)
-			)
-		)
-		(property "Description" ""
-			(at 220.98 41.91 0)
-			(effects
-				(font
-					(size 1.27 1.27)
-				)
-				(hide yes)
-			)
-		)
-		(property "LCSC Part" "C6931652"
-			(at 220.98 57.15 0)
-			(effects
-				(font
-					(size 1.27 1.27)
-				)
-				(hide yes)
-			)
-		)
-		(pin "6"
-		)
-		(pin "1"
-		)
-		(pin "4"
-		)
-		(pin "3"
-		)
-		(instances
-			(project ""
-				(path "/ad933f83-dd94-4dcc-b4f2-96fd54138c43"
-					(reference "U4")
-					(unit 1)
-				)
-			)
-		)
-	)
-	(symbol
 		(lib_id "Device:C_Small")
 		(at 199.39 199.39 0)
@@
 			)
 		)
-		(property "Mouser" "595-PCM5142PWR"
+		(property "Mouser" " 595-PCM5122PWR "
 			(at 72.39 180.34 0)
 			(effects
@@
 			)
 		)
+		(property "Mouser" " 603-CC1206JKX78BB225 "
+			(at 100.33 187.96 90)
+			(effects
+				(font
+					(size 1.27 1.27)
+				)
+				(hide yes)
+			)
+		)
 		(pin "2"
 		)
@@
 			)
 		)
-		(property "Mouser" "595-PCM5142PWR"
+		(property "Mouser" " 595-PCM5122PWR "
 			(at 160.02 179.07 0)
 			(effects
@@
 			)
 		)
+		(property "Mouser" " 603-CC1206JKX78BB225 "
+			(at 257.81 207.01 0)
+			(effects
+				(font
+					(size 1.27 1.27)
+				)
+				(hide yes)
+			)
+		)
 		(pin "2"
 		)
@@
 			)
 		)
+		(property "Mouser" " 603-CC1206JKX78BB225 "
+			(at 187.96 186.69 90)
+			(effects
+				(font
+					(size 1.27 1.27)
+				)
+				(hide yes)
+			)
+		)
 		(pin "2"
 		)
@@
 	)
 	(symbol
+		(lib_id "easyeda2kicad:DA101C_C6931652")
+		(at 220.98 41.91 0)
+		(unit 1)
+		(exclude_from_sim no)
+		(in_bom yes)
+		(on_board yes)
+		(dnp no)
+		(fields_autoplaced yes)
+		(property "Reference" "U6"
+			(at 220.9846 31.75 0)
+			(effects
+				(font
+					(size 1.27 1.27)
+				)
+			)
+		)
+		(property "Value" "DA101C_C6931652"
+			(at 220.9846 34.29 0)
+			(effects
+				(font
+					(size 1.27 1.27)
+				)
+			)
+		)
+		(property "Footprint" "easyeda2kicad:XFMR-TH_4P-L9.5-W9.0-P5.08-LS10.2_C9900096976"
+			(at 220.98 54.61 0)
+			(effects
+				(font
+					(size 1.27 1.27)
+				)
+				(hide yes)
+			)
+		)
+		(property "Datasheet" ""
+			(at 220.98 41.91 0)
+			(effects
+				(font
+					(size 1.27 1.27)
+				)
+				(hide yes)
+			)
+		)
+		(property "Description" ""
+			(at 220.98 41.91 0)
+			(effects
+				(font
+					(size 1.27 1.27)
+				)
+				(hide yes)
+			)
+		)
+		(property "LCSC Part" "C6931652"
+			(at 220.98 57.15 0)
+			(effects
+				(font
+					(size 1.27 1.27)
+				)
+				(hide yes)
+			)
+		)
+		(pin "4"
+		)
+		(pin "6"
+		)
+		(pin "3"
+		)
+		(pin "1"
+		)
+		(instances
+			(project ""
+				(path "/ad933f83-dd94-4dcc-b4f2-96fd54138c43"
+					(reference "U6")
+					(unit 1)
+				)
+			)
+		)
+	)
+	(symbol
 		(lib_id "Device:C_Small")
 		(at 86.36 74.93 0)
@@
 			)
 		)
+		(property "Mouser" " 603-CC1206JKX78BB225 "
+			(at 90.17 218.44 0)
+			(effects
+				(font
+					(size 1.27 1.27)
+				)
+				(hide yes)
+			)
+		)
 		(pin "2"
 		)
@@
 			)
 		)
+		(property "Mouser" " 603-CC1206JKX78BB225 "
+			(at 264.16 187.96 90)
+			(effects
+				(font
+					(size 1.27 1.27)
+				)
+				(hide yes)
+			)
+		)
 		(pin "2"
 		)
@@
 			)
 		)
-		(property "Mouser" "595-PCM5142PWR"
+		(property "Mouser" " 595-PCM5122PWR "
 			(at 237.49 180.34 0)
 			(effects
@@
 			)
 		)
-		(property "Value" "AMS1117-3.3"
+		(property "Value" "ZLDO1117QG33TA"
 			(at 76.2 68.58 0)
 			(effects
@@
 			(at 180.34 208.28 0)
 			(effects
+				(font
+					(size 1.27 1.27)
+				)
+				(hide yes)
+			)
+		)
+		(property "Mouser" " 603-CC1206JKX78BB225 "
+			(at 180.34 208.28 0)
+			(effects
