File: pcbs/dsp/0.1/dsp.kicad_pcb (KiCad board)
At the start: 4 copper layers, 85 x 55 mm, 48 parts, among them J1 Conn_01x04_Pin, J10 Conn_01x02_Pin, J2 Conn_01x03_Pin, J3 Conn_01x04_Pin, J4 Conn_01x04_Pin, J5 Conn_02x03_Odd_Even, J6 Conn_01x06_Pin, J7 Conn_01x02_Pin, J8 Conn_01x06_Pin, J9 Conn_01x04_Pin, U1 ESP32-S3-WROOM-1, U2 ESP32-S3-WROOM-1, U3 PI6CV304, U4 PI6CV304, U5 PI6CV304, U6 ESP32-S3-WROOM-1

Commit message: Updating readmes
Parts:
- added C9: 0.1u, Capacitor_SMD:C_0603_1608Metric_Pad1.08x0.95mm_HandSolder, F.Cu at (97.8, 70.3)
- added U6: TMP100, Package_TO_SOT_SMD:SOT-23-6, F.Cu at (97.9, 67.3)
- renumbered C4 to C1, C2 to C10, C3 to C11, C8 to C2, C5 to C3, C6 to C4, C7 to C5, C1 to C6, C10 to C7, C9 to C8, D2 to D1, D4 to D2, D1 to D4, H3 to H2, H2 to H3, J8 to J1, J7 to J10, J3 to J2, J9 to J3, J1 to J4, J10 to J6, J4 to J7, J6 to J8, J2 to J9, R13 to R1, R7 to R10, R14 to R11, R5 to R13, R1 to R14, R9 to R2, R6 to R3, R3 to R4, R10 to R5, R2 to R6, R11 to R7, R4 to R9, U3 to U2, U4 to U3, U5 to U4, U6 to U5, U2 to U7
Routing:
- net I2S_OUT_MCLK: track 41.5 -> 69.6 mm
- net I2S_LRCLK: track 111.4 -> 84.1 mm
- net 3V3: track 31.2 -> 37.4 mm
- net SDA: track 128.6 -> 134.7 mm, vias 3 -> 4
- net SCL: track 129.9 -> 133.9 mm, vias 3 -> 4
- net ADDR: track 103.3 -> 104.4 mm

Commit message: Updates to pcbs
Parts:
- R4, R6, R9: footprint Resistor_SMD:R_0603_1608Metric -> Resistor_SMD:R_0805_2012Metric
