File: pcbs/dsp/0.1/dsp.kicad_sch (KiCad schematic)
At the start: 48 parts, among them J1 Conn_01x04_Pin, J10 Conn_01x02_Pin, J2 Conn_01x03_Pin, J3 Conn_01x04_Pin, J4 Conn_01x04_Pin, J5 Conn_02x03_Odd_Even, J6 Conn_01x06_Pin, J7 Conn_01x02_Pin, J8 Conn_01x06_Pin, J9 Conn_01x04_Pin, U1 ESP32-S3-WROOM-1, U2 ESP32-S3-WROOM-1, U3 PI6CV304, U4 PI6CV304, U5 PI6CV304, U6 ESP32-S3-WROOM-1

Commit message: Updating readmes
Parts:
- added C9: 0.1u, Capacitor_SMD:C_0603_1608Metric_Pad1.08x0.95mm_HandSolder, symbol Device:C_Small
- added U6: TMP100, Package_TO_SOT_SMD:SOT-23-6, symbol Sensor_Temperature:TMP100
- renumbered C4 to C1, C2 to C10, C3 to C11, C8 to C2, C5 to C3, C6 to C4, C7 to C5, C1 to C6, C10 to C7, C9 to C8, D2 to D1, D4 to D2, D1 to D4, H3 to H2, H2 to H3, J8 to J1, J7 to J10, J3 to J2, J9 to J3, J1 to J4, J10 to J6, J4 to J7, J6 to J8, J2 to J9, R13 to R1, R7 to R10, R14 to R11, R5 to R13, R1 to R14, R9 to R2, R6 to R3, R3 to R4, R10 to R5, R2 to R6, R11 to R7, R4 to R9, U3 to U2, U4 to U3, U5 to U4, U6 to U5, U2 to U7
Connections:
- net 3V3: now also C9.1, U6.4 (V+)
- net GND: now also C9.2, U6.2 (GND), U6.3 (ADD1)
- net SCL: now also U6.1 (SCL)
- net SDA: now also U6.6 (SDA)
Other:
- moved on the sheet: C3, C4, C5, R2, R5, R7, U2, U3, U4

Commit message: Updates to pcbs
Parts:
- R4, R9: footprint Resistor_SMD:R_0603_1608Metric -> Resistor_SMD:R_0805_2012Metric; Mouser (none) -> 603-RT0805FRE0722RL
- R6: footprint Resistor_SMD:R_0603_1608Metric -> Resistor_SMD:R_0805_2012Metric; Field6 (none) -> 603-RT0805FRE0722RL
Changed lines of the file:
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@@
 			)
 		)
-		(property "Footprint" "Resistor_SMD:R_0603_1608Metric"
+		(property "Footprint" "Resistor_SMD:R_0805_2012Metric"
 			(at 182.88 224.79 0)
 			(effects
@@
 			)
 		)
+		(property "Mouser" "603-RT0805FRE0722RL "
+			(at 182.88 224.79 90)
+			(effects
+				(font
+					(size 1.27 1.27)
+				)
+				(hide yes)
+			)
+		)
 		(pin "2"
 		)
@@
 			)
 		)
-		(property "Footprint" "Resistor_SMD:R_0603_1608Metric"
+		(property "Footprint" "Resistor_SMD:R_0805_2012Metric"
 			(at 542.29 231.14 0)
 			(effects
@@
 			)
 		)
+		(property "Mouser" " 603-RT0805FRE0722RL "
+			(at 542.29 231.14 90)
+			(effects
+				(font
+					(size 1.27 1.27)
+				)
+				(hide yes)
+			)
+		)
 		(pin "2"
 		)
@@
 			)
 		)
-		(property "Footprint" "Resistor_SMD:R_0603_1608Metric"
+		(property "Footprint" "Resistor_SMD:R_0805_2012Metric"
 			(at 349.25 224.79 0)
 			(effects
@@
 			(effects
 				(font
+					(size 1.27 1.27)
+				)
+				(hide yes)
+			)
+		)
+		(property "Mouser" ""
+			(at 349.25 224.79 90)
+			(effects
+				(font
+					(size 1.27 1.27)
+				)
+				(hide yes)
+			)
+		)
+		(property "Field6" "603-RT0805FRE0722RL "
+			(at 349.25 224.79 90)
+			(effects
+				(font
