File: pcbs/extend/1.0/extend.kicad_sch (KiCad schematic)
At the start: 25 parts, among them J1 Conn_01x02_Male, J10 Conn_01x02_Male, J11 Conn_01x02_Pin, J12 Conn_01x03_Pin, J2 Conn_01x05_Pin, J3 Conn_01x04_Pin, J4 Conn_01x06_Pin, J5 Conn_01x02_Male, J6 Conn_01x02_Male, J7 Conn_01x04_Pin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

Commit message: Updates to pcbs
Parts:
- U1: Mouser (none) -> 579-MCP23017-E/SS
Changed lines of the file:
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@@
+			)
+		)
+		(property "Mouser" " 579-MCP23017-E/SS "
+			(at 254 69.85 0)
+			(effects
+				(font
+					(size 1.27 1.27)
+				)
+				(hide yes)
 			)
 		)
