File: pcbs/mono/1.0/mono.kicad_pcb (KiCad board)
At the start: 2 copper layers, 100 x 45 mm, 36 parts, among them J1 Conn_01x03_Male, J10 Conn_01x02_Pin, J11 Conn_01x02_Pin, J12 Conn_01x02_Pin, J13 Conn_01x03_Pin, J2 Conn_01x02_Pin, J3 Conn_01x02_Pin, J5 Conn_01x04_Pin, J6 Conn_01x03_Male, J7 Conn_01x03_Male, J8 Conn_01x02_Pin, J9 Conn_01x02_Pin, Q1 BC807, Q2 BC817K-40, Q3 BC817K-40, U1 TMP100

Commit message: Updates to pcbs
Parts:
- removed the J2 at (154.4, 77.0)
- removed the J3 at (161.7, 77.0)
- added D2: RED, LED_SMD:LED_0603_1608Metric_Pad1.05x0.95mm_HandSolder, F.Cu at (179.2, 83.3)
- added J1: Conn_01x03_Pin, Connector_JST:JST_PH_B3B-PH-K_1x03_P2.00mm_Vertical, F.Cu at (156.4, 76.9)
- added R2: 300R, Resistor_SMD:R_0603_1608Metric_Pad0.98x0.95mm_HandSolder, F.Cu at (175.6, 83.3)
- added R5: 550R, Resistor_SMD:R_0603_1608Metric_Pad0.98x0.95mm_HandSolder, F.Cu at (181.6, 88.6)
- added R6: 150R, Resistor_SMD:R_0603_1608Metric_Pad0.98x0.95mm_HandSolder, F.Cu at (184.7, 88.6)
- R10: renamed from R6; value 10K -> 50K
- R9: renamed from R5; value 90K -> 100K
- moved D1 51.6 mm to (179.2, 81.0)
- moved R1 51.6 mm to (175.6, 81.0)
- moved J9 0.10 mm to (161.7, 116.1)
- renumbered J11 to J10, J10 to J11, J1 to J2, J13 to J3, J12 to J4, J7 to J6, J6 to J7, J9 to J8, J8 to J9, Q3 to Q2, Q2 to Q3, R8 to R1, R7 to R11, R9 to R12, R1 to R3, R2 to R4, R3 to R7, R4 to R8
Connections:
- J3 pad 1: ACTIVE_IN -> LED_ACTIVE
- J3 pad 3: ACTIVE_NEG -> LED_STANDBY
Routing:
- net 3V3: track 96.8 -> 69.5 mm, vias 5 -> 7
- net ACTIVE_IN: track 16.3 -> 34.1 mm, vias 2 -> 5
- net PGND: track 176.0 -> 159.7 mm, vias 7 -> 9
- net LED_ACTIVE: track 0.00 -> 8.88 mm
- net LED_STANDBY: track 0.00 -> 5.15 mm
- net ACTIVE_NEG: track 19.3 -> 21.2 mm, vias 0 -> 2
- net Net-(D2-A): track 0.00 -> 1.81 mm
- net WOOFER: track 39.0 -> 40.5 mm
- net TWEETER: track 39.0 -> 39.9 mm
- net AGND: vias 2 -> 3
Other:
- board text added: "ACTIVE"
- board text added: "TWEET/WOOF"
- board text removed: "TWEET_IN"
- board text removed: "WOOF_IN"
