File: pcbs/mono/1.0/mono.kicad_sch (KiCad schematic)
At the start: 36 parts, among them J1 Conn_01x03_Male, J10 Conn_01x02_Pin, J11 Conn_01x02_Pin, J12 Conn_01x02_Pin, J13 Conn_01x03_Pin, J2 Conn_01x02_Pin, J3 Conn_01x02_Pin, J5 Conn_01x04_Pin, J6 Conn_01x03_Male, J7 Conn_01x03_Male, J8 Conn_01x02_Pin, J9 Conn_01x02_Pin, Q1 BC807, Q2 BC817K-40, Q3 BC817K-40, U1 TMP100

Commit message: Updates to pcbs
Parts:
- removed J2, J3: Conn_01x02_Pin, Connector_JST:JST_PH_B2B-PH-K_1x02_P2.00mm_Vertical, symbol Connector:Conn_01x02_Pin
- added D2: RED, LED_SMD:LED_0603_1608Metric_Pad1.05x0.95mm_HandSolder, symbol Device:LED
- added J1: Conn_01x03_Pin, Connector_JST:JST_PH_B3B-PH-K_1x03_P2.00mm_Vertical, symbol Connector:Conn_01x03_Pin
- added R2: 300R, Resistor_SMD:R_0603_1608Metric_Pad0.98x0.95mm_HandSolder, symbol Device:R_Small
- added R5: 550R, Resistor_SMD:R_0603_1608Metric_Pad0.98x0.95mm_HandSolder, symbol Device:R_Small
- added R6: 150R, Resistor_SMD:R_0603_1608Metric_Pad0.98x0.95mm_HandSolder, symbol Device:R_Small
- R10: renamed from R6; value 10K -> 50K
- R9: renamed from R5; value 90K -> 100K
- renumbered J11 to J10, J10 to J11, J1 to J2, J13 to J3, J12 to J4, J7 to J6, J6 to J7, J9 to J8, J8 to J9, Q3 to Q2, Q2 to Q3, R8 to R1, R7 to R11, R9 to R12, R1 to R3, R2 to R4, R3 to R7, R4 to R8
Connections:
- net ACTIVE_IN: now also R2.2, R5.2; no longer J3.1 (Pin_1)
- net ACTIVE_NEG: now also R6.2; no longer J3.3 (Pin_3)
- net AGND: now also J1.2 (Pin_2)
- net PGND: now also D2.1 (K)
- net TWEETER: now also J1.3 (Pin_3)
- net WOOFER: now also J1.1 (Pin_1)
- new net: D2.2 (A), R2.1
- new net LED_ACTIVE: J3.1 (Pin_1), R5.1
- new net LED_STANDBY: J3.3 (Pin_3), R6.1
