File: pcbs/spdif/1.0/spdif.kicad_pcb (KiCad board)
At the start: 4 copper layers, 85 x 55 mm, 67 parts, among them J1 Conn_01x04_Pin, J10 Conn_01x02_Pin, J11 Conn_01x03_Pin, J12 Conn_01x04_Pin, J13 Conn_01x04_Pin, J14 Conn_01x05_Pin, J2 Conn_01x04_Pin, J3 Conn_01x02_Pin, J4 Conn_01x02_Pin, J5 Conn_01x02_Pin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

Commit message: Updates to pcbs
Parts:
- C14: footprint Capacitor_SMD:C_0603_1608Metric -> Capacitor_SMD:C_1206_3216Metric
- R2, R3, R4, R5: footprint Resistor_SMD:R_0603_1608Metric -> Resistor_SMD:R_0805_2012Metric
- moved C14 0.61 mm to (69.9, 58.6)
Routing:
- net Net-(C14-Pad2): track 1.55 -> 2.41 mm
- net FILTGND: track 6.55 -> 7.29 mm
