File: pcbs/_ready/inputs/1.0/inputs.kicad_pcb (KiCad board)
At the start: 2 copper layers, 85 x 55 mm, 23 parts, among them J1 Conn_01x03_Pin, J10 Conn_01x03_Pin, J11 Conn_01x03_Pin, J12 Conn_01x03_Pin, J13 Conn_01x02_Pin, J2 Conn_01x03_Pin, J3 Conn_01x03_Pin, J4 Conn_01x03_Pin, J5 Conn_01x03_Pin, J6 Conn_01x03_Pin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

Commit message: More work on PCBs
Changed lines of the file:
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@@
 		(property "Reference" "J6"
 			(at 2 -2.9 0)
+			(unlocked yes)
 			(layer "F.SilkS")
 			(hide yes)
 			(effects
 				(font
-					(size 1 1)
-					(thickness 0.15)
+					(size 0.8 0.8)
+					(thickness 0.1)
 				)
 			)
@@
 		(property "Reference" "H1"
 			(at 0 -3.8 90)
+			(unlocked yes)
 			(layer "F.SilkS")
 			(hide yes)
 			(effects
 				(font
-					(size 1 1)
-					(thickness 0.15)
+					(size 0.8 0.8)
+					(thickness 0.1)
 				)
 			)
@@
 		(property "Reference" "H3"
 			(at 0 -3.8 90)
+			(unlocked yes)
 			(layer "F.SilkS")
 			(hide yes)
 			(effects
 				(font
-					(size 1 1)
-					(thickness 0.15)
+					(size 0.8 0.8)
+					(thickness 0.1)
 				)
 			)
@@
 		(property "Reference" "J4"
 			(at 2 -2.9 0)
+			(unlocked yes)
 			(layer "F.SilkS")
 			(hide yes)
 			(effects
 				(font
-					(size 1 1)
-					(thickness 0.15)
+					(size 0.8 0.8)
+					(thickness 0.1)
 				)
 			)
@@
 		(property "Reference" "H2"
 			(at 0 -3.8 90)
+			(unlocked yes)
 			(layer "F.SilkS")
 			(hide yes)
 			(effects
 				(font
-					(size 1 1)
-					(thickness 0.15)
+					(size 0.8 0.8)
+					(thickness 0.1)
 				)
 			)
@@
 		(property "Reference" "J3"
 			(at 2 -2.9 0)
+			(unlocked yes)
 			(layer "F.SilkS")
 			(hide yes)
 			(effects
 				(font
-					(size 1 1)
-					(thickness 0.15)
+					(size 0.8 0.8)
+					(thickness 0.1)
 				)
 			)
@@
 		(property "Reference" "J12"
 			(at 2 -2.9 0)
+			(unlocked yes)
 			(layer "F.SilkS")
 			(hide yes)
 			(effects
 				(font
-					(size 1 1)
-					(thickness 0.15)
+					(size 0.8 0.8)
+					(thickness 0.1)
 				)
 			)
@@
 		(property "Reference" "C5"
 			(at 0 -1.85 90)
+			(unlocked yes)
 			(layer "F.SilkS")
 			(effects
 				(font
-					(size 1 1)
-					(thickness 0.15)
+					(size 0.8 0.8)
+					(thickness 0.1)
 				)
 			)
@@
 		(property "Reference" "J2"
 			(at 2 -2.9 0)
+			(unlocked yes)
 			(layer "F.SilkS")
 			(hide yes)
 			(effects
 				(font
-					(size 1 1)
-					(thickness 0.15)
+					(size 0.8 0.8)
+					(thickness 0.1)
 				)
 			)
@@
 		(property "Reference" "C2"
 			(at 0 -1.85 90)
+			(unlocked yes)
 			(layer "F.SilkS")
 			(effects
 				(font
-					(size 1 1)
-					(thickness 0.15)
+					(size 0.8 0.8)
+					(thickness 0.1)
 				)
 			)
@@
 		(property "Reference" "J10"
 			(at 2 -2.9 0)
+			(unlocked yes)
 			(layer "F.SilkS")
 			(hide yes)
 			(effects
 				(font
-					(size 1 1)
-					(thickness 0.15)
+					(size 0.8 0.8)
+					(thickness 0.1)
 				)
 			)
@@
 		(property "Reference" "C4"
 			(at 0 -1.85 90)
+			(unlocked yes)
 			(layer "F.SilkS")
 			(effects
 				(font
-					(size 1 1)
-					(thickness 0.15)
+					(size 0.8 0.8)
+					(thickness 0.1)
 				)
 			)
@@
 		(property "Reference" "J5"
 			(at 2 -2.9 0)
+			(unlocked yes)
 			(layer "F.SilkS")
 			(hide yes)
 			(effects
 				(font
-					(size 1 1)
-					(thickness 0.15)
+					(size 0.8 0.8)
+					(thickness 0.1)
 				)
 			)
@@
 		(property "Reference" "C3"
 			(at 0 -1.85 90)
+			(unlocked yes)
 			(layer "F.SilkS")
 			(effects
 				(font
-					(size 1 1)
-					(thickness 0.15)
+					(size 0.8 0.8)
+					(thickness 0.1)
 				)
 			)
@@
 		(property "Reference" "C1"
 			(at 0 -1.85 90)
+			(unlocked yes)
 			(layer "F.SilkS")
 			(effects
 				(font
-					(size 1 1)
-					(thickness 0.15)
+					(size 0.8 0.8)
+					(thickness 0.1)
 				)
 			)
@@
 		(property "Reference" "J11"
 			(at 2 -2.9 0)
+			(unlocked yes)
 			(layer "F.SilkS")
 			(hide yes)
 			(effects
 				(font
-					(size 1 1)
-					(thickness 0.15)
+					(size 0.8 0.8)
+					(thickness 0.1)
 				)
 			)
@@
 		(property "Reference" "J9"
 			(at 2 -2.9 0)
+			(unlocked yes)
 			(layer "F.SilkS")
 			(hide yes)
 			(effects
 				(font
-					(size 1 1)
-					(thickness 0.15)
+					(size 0.8 0.8)
+					(thickness 0.1)
 				)
 			)
@@
 		(property "Reference" "H4"
 			(at 0 -3.8 90)
+			(unlocked yes)
 			(layer "F.SilkS")
 			(hide yes)
 			(effects
 				(font
-					(size 1 1)
-					(thickness 0.15)
+					(size 0.8 0.8)
+					(thickness 0.1)
 				)
 			)
@@
 		(property "Reference" "J8"
 			(at 2 -2.9 0)
+			(unlocked yes)
 			(layer "F.SilkS")
 			(hide yes)
 			(effects
 				(font
-					(size 1 1)
-					(thickness 0.15)
+					(size 0.8 0.8)
+					(thickness 0.1)
 				)
 			)
@@
 		(property "Reference" "J1"
 			(at 2 -2.9 0)
+			(unlocked yes)
 			(layer "F.SilkS")
 			(hide yes)
 			(effects
 				(font
-					(size 1 1)
-					(thickness 0.15)
+					(size 0.8 0.8)
+					(thickness 0.1)
 				)
 			)
@@
 		(property "Reference" "J7"
 			(at 2 -2.9 0)
+			(unlocked yes)
 			(layer "F.SilkS")
 			(hide yes)
 			(effects
 				(font
-					(size 1 1)
-					(thickness 0.15)
+					(size 0.8 0.8)
+					(thickness 0.1)
 				)
 			)
@@
 		(property "Reference" "J13"
 			(at 1.98 -4.9 90)
+			(unlocked yes)
 			(layer "F.SilkS")
 			(hide yes)
 			(effects
 				(font
-					(size 1 1)
-					(thickness 0.15)
+					(size 0.8 0.8)
+					(thickness 0.1)
 				)
 			)
@@
 		(property "Reference" "C6"
 			(at 0 -1.85 90)
+			(unlocked yes)
 			(layer "F.SilkS")
 			(effects
 				(font
-					(size 1 1)
-					(thickness 0.15)
+					(size 0.8 0.8)
+					(thickness 0.1)
 				)
 			)
@@
 		)
 	)
+	(gr_rect
+		(start 158.9 64.1)
+		(end 163.9 69.1)
+		(stroke
+			(width 0.1)
+			(type solid)
+		)
+		(fill solid)
+		(layer "F.SilkS")
+	)
 	(gr_line
