File: pcbs/_ready/psu/1.0/_autosave-psu.kicad_sch (KiCad schematic)
At the start: 35 parts, among them J1 Conn_01x02_Male, J2 Conn_01x03_Male, J3 Conn_01x02_Pin, J4 Conn_01x03_Male, J5 Conn_01x03_Male, J6 Conn_01x03_Male, J7 Conn_01x02_Pin, J8 Conn_01x02_Male, U1 INA260, U2 INA260

Commit message: More work on PCBs
Parts:
- C3, C6: footprint Capacitor_THT:CP_Radial_D16.0mm_P7.50mm -> Capacitor_THT:CP_Radial_D18.0mm_P7.50mm
Changed lines of the file:
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@@
 			)
 		)
-		(property "Footprint" "Capacitor_THT:CP_Radial_D16.0mm_P7.50mm"
+		(property "Footprint" "Capacitor_THT:CP_Radial_D18.0mm_P7.50mm"
 			(at 82.55 78.74 0)
 			(effects
@@
 			)
 		)
-		(property "Footprint" "Capacitor_THT:CP_Radial_D16.0mm_P7.50mm"
+		(property "Footprint" "Capacitor_THT:CP_Radial_D18.0mm_P7.50mm"
 			(at 82.55 97.79 0)
 			(effects
