File: pcbs/_ready/psu/1.0/psu.kicad_pcb (KiCad board)
At the start: 2 copper layers, 95 x 95 mm, 35 parts, among them J1 Conn_01x02_Male, J2 Conn_01x03_Male, J3 Conn_01x02_Pin, J4 Conn_01x03_Male, J5 Conn_01x03_Male, J6 Conn_01x03_Male, J7 Conn_01x02_Pin, J8 Conn_01x02_Male, U1 INA260, U2 INA260

Commit message: More work on PCBs
Changed lines of the file:
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@@
 		(property ki_fp_filters "CP_*")
 		(sheetname "Root")
-		(sheetfile "PSU.kicad_sch")
+		(sheetfile "psu.kicad_sch")
 		(attr through_hole)
 		(fp_line
@@
 		(property ki_fp_filters "MountingHole*")
 		(sheetname "Root")
-		(sheetfile "PSU.kicad_sch")
+		(sheetfile "psu.kicad_sch")
 		(attr exclude_from_pos_files)
 		(fp_circle
@@
 		(property ki_fp_filters "LED* LED_SMD:* LED_THT:*")
 		(sheetname "Root")
-		(sheetfile "PSU.kicad_sch")
+		(sheetfile "psu.kicad_sch")
 		(attr smd)
 		(fp_line
@@
 		(property ki_fp_filters "CP_*")
 		(sheetname "Root")
-		(sheetfile "PSU.kicad_sch")
+		(sheetfile "psu.kicad_sch")
 		(attr through_hole)
 		(fp_line
@@
 		(property ki_fp_filters "Connector*:*_1x??_*")
 		(sheetname "Root")
-		(sheetfile "PSU.kicad_sch")
+		(sheetfile "psu.kicad_sch")
 		(attr through_hole)
 		(fp_line
@@
 		(property ki_fp_filters "R_*")
 		(sheetname "Root")
-		(sheetfile "PSU.kicad_sch")
+		(sheetfile "psu.kicad_sch")
 		(attr smd)
 		(fp_line
@@
 		(property ki_fp_filters "Connector*:*_1x??_*")
 		(sheetname "Root")
-		(sheetfile "PSU.kicad_sch")
+		(sheetfile "psu.kicad_sch")
 		(attr through_hole)
 		(fp_line
@@
 		(property ki_fp_filters "MountingHole*")
 		(sheetname "Root")
-		(sheetfile "PSU.kicad_sch")
+		(sheetfile "psu.kicad_sch")
 		(attr exclude_from_pos_files)
 		(fp_circle
@@
 		(property ki_fp_filters "R_*")
 		(sheetname "Root")
-		(sheetfile "PSU.kicad_sch")
+		(sheetfile "psu.kicad_sch")
 		(attr smd)
 		(fp_line
@@
 		(property ki_fp_filters "CP_*")
 		(sheetname "Root")
-		(sheetfile "PSU.kicad_sch")
+		(sheetfile "psu.kicad_sch")
 		(attr through_hole)
 		(fp_line
@@
 		)
 		(sheetname "Root")
-		(sheetfile "PSU.kicad_sch")
+		(sheetfile "psu.kicad_sch")
 		(attr smd)
 		(fp_line
@@
 		(property ki_fp_filters "Connector*:*_1x??_*")
 		(sheetname "Root")
-		(sheetfile "PSU.kicad_sch")
+		(sheetfile "psu.kicad_sch")
 		(attr through_hole)
 		(fp_line
@@
 		(property ki_fp_filters "LED* LED_SMD:* LED_THT:*")
 		(sheetname "Root")
-		(sheetfile "PSU.kicad_sch")
+		(sheetfile "psu.kicad_sch")
 		(attr smd)
 		(fp_line
@@
 		(property ki_fp_filters "R_*")
 		(sheetname "Root")
-		(sheetfile "PSU.kicad_sch")
+		(sheetfile "psu.kicad_sch")
 		(attr smd)
 		(fp_line
@@
 		(property ki_fp_filters "LED* LED_SMD:* LED_THT:*")
 		(sheetname "Root")
-		(sheetfile "PSU.kicad_sch")
+		(sheetfile "psu.kicad_sch")
 		(attr smd)
 		(fp_line
@@
 		(property ki_fp_filters "C_*")
 		(sheetname "Root")
-		(sheetfile "PSU.kicad_sch")
+		(sheetfile "psu.kicad_sch")
 		(attr smd)
 		(fp_line
@@
 		(property ki_fp_filters "Connector*:*_1x??_*")
 		(sheetname "Root")
-		(sheetfile "PSU.kicad_sch")
+		(sheetfile "psu.kicad_sch")
 		(attr through_hole)
 		(fp_line
@@
 		(property ki_fp_filters "LED* LED_SMD:* LED_THT:*")
 		(sheetname "Root")
-		(sheetfile "PSU.kicad_sch")
+		(sheetfile "psu.kicad_sch")
 		(attr smd)
 		(fp_line
@@
 		(property ki_fp_filters "CP_*")
 		(sheetname "Root")
-		(sheetfile "PSU.kicad_sch")
+		(sheetfile "psu.kicad_sch")
 		(attr through_hole)
 		(fp_line
@@
 		(property ki_fp_filters "Connector*:*_1x??_*")
 		(sheetname "Root")
-		(sheetfile "PSU.kicad_sch")
+		(sheetfile "psu.kicad_sch")
 		(attr through_hole)
 		(fp_line
@@
 		(property ki_fp_filters "Connector*:*_1x??_*")
 		(sheetname "Root")
-		(sheetfile "PSU.kicad_sch")
+		(sheetfile "psu.kicad_sch")
 		(attr through_hole)
 		(fp_line
@@
 		(property ki_fp_filters "C_*")
 		(sheetname "Root")
-		(sheetfile "PSU.kicad_sch")
+		(sheetfile "psu.kicad_sch")
 		(attr smd)
 		(fp_line
@@
 		(property ki_fp_filters "SM*")
 		(sheetname "Root")
-		(sheetfile "PSU.kicad_sch")
+		(sheetfile "psu.kicad_sch")
 		(attr through_hole)
 		(fp_rect
@@
 		(property ki_fp_filters "CP_*")
 		(sheetname "Root")
-		(sheetfile "PSU.kicad_sch")
+		(sheetfile "psu.kicad_sch")
 		(attr through_hole)
 		(fp_line
@@
 		(property ki_fp_filters "Connector*:*_1x??_*")
 		(sheetname "Root")
-		(sheetfile "PSU.kicad_sch")
+		(sheetfile "psu.kicad_sch")
 		(attr through_hole)
 		(fp_line
@@
 		(property ki_fp_filters "R_*")
 		(sheetname "Root")
-		(sheetfile "PSU.kicad_sch")
+		(sheetfile "psu.kicad_sch")
 		(attr smd)
 		(fp_line
@@
 		(property ki_fp_filters "MountingHole*")
 		(sheetname "Root")
-		(sheetfile "PSU.kicad_sch")
+		(sheetfile "psu.kicad_sch")
 		(attr exclude_from_pos_files)
 		(fp_circle
@@
 		(property ki_fp_filters "C_*")
 		(sheetname "Root")
-		(sheetfile "PSU.kicad_sch")
+		(sheetfile "psu.kicad_sch")
 		(attr smd)
 		(fp_line
@@
 		(property ki_fp_filters "Connector*:*_1x??_*")
 		(sheetname "Root")
-		(sheetfile "PSU.kicad_sch")
+		(sheetfile "psu.kicad_sch")
 		(attr through_hole)
 		(fp_line
@@
 		(property ki_fp_filters "SM*")
 		(sheetname "Root")
-		(sheetfile "PSU.kicad_sch")
+		(sheetfile "psu.kicad_sch")
 		(attr through_hole)
 		(fp_rect
@@
 		(property ki_fp_filters "R_*")
 		(sheetname "Root")
-		(sheetfile "PSU.kicad_sch")
+		(sheetfile "psu.kicad_sch")
 		(attr smd)
 		(fp_line
@@
 		)
 		(sheetname "Root")
-		(sheetfile "PSU.kicad_sch")
+		(sheetfile "psu.kicad_sch")
 		(attr smd)
 		(fp_line
@@
 		(property ki_fp_filters "CP_*")
 		(sheetname "Root")
-		(sheetfile "PSU.kicad_sch")
+		(sheetfile "psu.kicad_sch")
 		(attr through_hole)
 		(fp_line
@@
 		(property ki_fp_filters "R_*")
 		(sheetname "Root")
-		(sheetfile "PSU.kicad_sch")
+		(sheetfile "psu.kicad_sch")
 		(attr smd)
 		(fp_line
@@
 		(property ki_fp_filters "MountingHole*")
 		(sheetname "Root")
-		(sheetfile "PSU.kicad_sch")
+		(sheetfile "psu.kicad_sch")
 		(attr exclude_from_pos_files)
 		(fp_circle
@@
 		)
 	)
+	(gr_rect
+		(start 226.5 44.7)
+		(end 231.5 49.7)
+		(stroke
+			(width 0.1)
+			(type solid)
+		)
+		(fill solid)
+		(layer "F.SilkS")
+	)
 	(gr_line
